Commit message: Replace pkg name in all files

File: jsk_2014_baxter_apc/config/baxter_white_hand.urdf (robot description, URDF)
Before this commit: robot baxter, 54 links, 53 joints
Links:
- link custom_vacuum_link: geometry collision cylinder length=0.45 radius=0.02; visual mesh filename=package://jsk_2014_baxter_apc/config/mesh/long1_simple.dae scale=0.001 0.001 0.001
- link custom_vacuum_link_base: geometry collision cylinder length=0.01 radius=0.04; visual mesh filename=package://jsk_2014_baxter_apc/config/mesh/jigukailong2_simp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 scale=0.001 0.001 0.001

File: jsk_2014_baxter_apc/config/baxter_white_hand.urdf.xacro (robot description, xacro)
@@ -13,5 +13,5 @@
       <origin rpy="0 0 1.57" xyz="0 0 -0.07"/>
       <geometry>
-        <mesh filename="package://jsk_2014_picking_challenge/config/mesh/long1_simple.dae" scale="0.001 0.001 0.001"/>
+        <mesh filename="package://jsk_2014_baxter_apc/config/mesh/long1_simple.dae" scale="0.001 0.001 0.001"/>
       </geometry>
       <material name="white">
@@ -28,5 +28,5 @@
     <visual>
       <geometry>
-        <mesh filename="package://jsk_2014_picking_challenge/config/mesh/light/jigu_long2_right_kari1.dae" scale="0.001 0.001 0.001"/>
+        <mesh filename="package://jsk_2014_baxter_apc/config/mesh/light/jigu_long2_right_kari1.dae" scale="0.001 0.001 0.001"/>
       </geometry>
       <material name="white">
@@ -44,5 +44,5 @@
       <origin rpy="0 0 1.57" xyz="0 0 -0.07"/>
       <geometry>
-        <mesh filename="package://jsk_2014_picking_challenge/config/mesh/long1_simple.dae" scale="0.001 0.001 0.001"/>
+        <mesh filename="package://jsk_2014_baxter_apc/config/mesh/long1_simple.dae" scale="0.001 0.001 0.001"/>
       </geometry>
       <material name="white">
@@ -59,5 +59,5 @@
     <visual>
       <geometry>
-        <mesh filename="package://jsk_2014_picking_challenge/config/mesh/light/jigu_long2_left_kari2.dae" scale="0.001 0.001 0.001"/>
+        <mesh filename="package://jsk_2014_baxter_apc/config/mesh/light/jigu_long2_left_kari2.dae" scale="0.001 0.001 0.001"/>
       </geometry>
       <material name="white">
