Commit message: Update Baxter urdf model for long vacuum hand

File: jsk_2015_05_baxter_apc/config/baxter_white_hand.urdf.xacro (robot description, xacro)
@@ -5,5 +5,5 @@
   <xacro:property name="width_base" value=".04" />
   <xacro:property name="width_side2_base" value=".035" />
-  <xacro:property name="bodylen" value=".14" />
+  <xacro:property name="bodylen" value=".45" />
   <xacro:property name="bodylen_base" value=".01" />
   <xacro:property name="bodylen_side" value=".15" />

Commit message: [config/baxter_white_hand.urdf.xacro] Update white hand pos

File: jsk_2015_05_baxter_apc/config/baxter_white_hand.urdf.xacro (robot description, xacro)
@@ -10,4 +10,5 @@
   <xacro:property name="bodylen_side2" value=".12" />
   <xacro:property name="bodylen_side2_base" value=".06" />
+  <xacro:property name="right_wrist_offset_x" value="-0.04" />
   <link name="custom_vacuum_link">
     <visual>
@@ -89,25 +90,25 @@
     <parent link="right_wrist"/>
     <child link="custom_vacuum_link"/>
-    <origin rpy="0 0 0" xyz="0 0 0.18" />
+    <origin rpy="0 0 0" xyz="${right_wrist_offset_x} 0 0.18" />
   </joint>
   <joint name="right_custom_joint_base" type="fixed">
     <parent link="right_wrist"/>
     <child link="custom_vacuum_link_base"/>
-    <origin rpy="0 0 1.57" xyz="0 0 0.11" />
+    <origin rpy="0 0 0" xyz="${right_wrist_offset_x} 0 0.11" />
   </joint>
   <joint name="right_custom_joint_side" type="fixed">
     <parent link="right_wrist"/>
     <child link="custom_vacuum_link_side"/>
-    <origin rpy="1.57 0 0" xyz="0 0.05 0.15" />
+    <origin rpy="1.57 0 0" xyz="${right_wrist_offset_x} 0 0.15" />
   </joint>
   <joint name="right_custom_joint_side2" type="fixed">
     <parent link="right_wrist"/>
     <child link="custom_vacuum_link_side2"/>
-    <origin rpy="0 0 0" xyz="0 0.1 0.08" />
+    <origin rpy="0 0 0" xyz="${right_wrist_offset_x} 0 0.08" />
   </joint>
   <joint name="right_custom_joint_side2_base" type="fixed">
     <parent link="right_wrist"/>
     <child link="custom_vacuum_link_side2_base"/>
-    <origin rpy="0 0 0" xyz="0 0.1 0.04" />
+    <origin rpy="0 0 0" xyz="${right_wrist_offset_x} 0 0.04" />
   </joint>
 </robot>

Commit message: [config/baxter_white_hand.urdf.xacro] cylidner with 0 may crash urdf_to_collada, use small box

File: jsk_2015_05_baxter_apc/config/baxter_white_hand.urdf.xacro (robot description, xacro)
@@ -45,5 +45,5 @@
     <visual>
       <geometry>
-        <cylinder radius="0" length="0"/>
+        <box size="0.001 0.001 0.001" />
       </geometry>
       <material name="white">
@@ -60,5 +60,5 @@
     <visual>
       <geometry>
-        <cylinder radius="0" length="0"/>
+        <box size="0.001 0.001 0.001" />
       </geometry>
       <material name="white">
@@ -83,5 +83,5 @@
     <collision>
       <geometry>
-        <cylinder radius="0" length="0"/>
+        <box size="0.001 0.001 0.001" />
       </geometry>
     </collision>

Commit message: [config/baxter_white_hand.urdf.xacro] use simple mesh model

File: jsk_2015_05_baxter_apc/config/baxter_white_hand.urdf.xacro (robot description, xacro)
@@ -1,5 +1,5 @@
 <?xml version="1.0"?>
 <robot xmlns:xacro="http://ros.org/wiki/xacro" name="baxter_custom_white">
-  <xacro:include filename="$(find baxter_description)/urdf/baxter.urdf" />
+  <xacro:include filename="$(find baxter_description)/urdf/baxter_simple.urdf" />
   <xacro:property name="width" value=".02" />
   <xacro:property name="width_base" value=".04" />
@@ -15,5 +15,5 @@
       <origin rpy="0 0 1.57" xyz="0 0 -0.07"/>
       <geometry>
-        <mesh filename="package://jsk_2014_picking_challenge/config/mesh/long1.dae" scale="0.001 0.001 0.001"/>
+        <mesh filename="package://jsk_2014_picking_challenge/config/mesh/long1_simple.dae" scale="0.001 0.001 0.001"/>
       </geometry>
       <material name="white">
@@ -30,5 +30,5 @@
     <visual>
       <geometry>
-        <mesh filename="package://jsk_2014_picking_challenge/config/mesh/jigukailong2.dae" scale="0.001 0.001 0.001"/>
+        <mesh filename="package://jsk_2014_picking_challenge/config/mesh/jigukailong2_simple.dae" scale="0.001 0.001 0.001"/>
       </geometry>
       <material name="white">

Commit message: Update Baxter URDF for dual arm

File: jsk_2015_05_baxter_apc/config/baxter_white_hand.urdf.xacro (robot description, xacro)
@@ -5,11 +5,9 @@
   <xacro:property name="width_base" value=".04" />
   <xacro:property name="width_side2_base" value=".035" />
-  <xacro:property name="bodylen" value=".45" />
+  <xacro:property name="bodylen" value=".49" />
   <xacro:property name="bodylen_base" value=".01" />
-  <xacro:property name="bodylen_side" value=".15" />
-  <xacro:property name="bodylen_side2" value=".12" />
-  <xacro:property name="bodylen_side2_base" value=".06" />
-  <xacro:property name="right_wrist_offset_x" value="-0.04" />
-  <link name="custom_vacuum_link">
+  <xacro:property name="right_wrist_offset_x" value="-0.01" />
+  <xacro:property name="left_wrist_offset_x" value="-0.01" />
+  <link name="right_custom_vacuum_link">
     <visual>
       <origin rpy="0 0 1.57" xyz="0 0 -0.07"/>
@@ -27,8 +25,8 @@
     </collision>
   </link>
-  <link name="custom_vacuum_link_base">
+  <link name="right_custom_vacuum_link_base">
     <visual>
       <geometry>
-        <mesh filename="package://jsk_2014_picking_challenge/config/mesh/jigukailong2_simple.dae" scale="0.001 0.001 0.001"/>
+        <mesh filename="package://jsk_2014_picking_challenge/config/mesh/light/jigu_long2_right_kari1.dae" scale="0.001 0.001 0.001"/>
       </geometry>
       <material name="white">
@@ -42,8 +40,9 @@
     </collision>
   </link>
-  <link name="custom_vacuum_link_side">
+  <link name="left_custom_vacuum_link">
     <visual>
+      <origin rpy="0 0 1.57" xyz="0 0 -0.07"/>
       <geometry>
-        <box size="0.001 0.001 0.001" />
+        <mesh filename="package://jsk_2014_picking_challenge/config/mesh/long1_simple.dae" scale="0.001 0.001 0.001"/>
       </geometry>
       <material name="white">
@@ -53,12 +52,12 @@
     <collision>
       <geometry>
-        <cylinder radius="${width}" length="${bodylen_side}"/>
+        <cylinder radius="${width}" length="${bodylen}"/>
       </geometry>
     </collision>
   </link>
-  <link name="custom_vacuum_link_side2">
+  <link name="left_custom_vacuum_link_base">
     <visual>
       <geometry>
-        <box size="0.001 0.001 0.001" />
+        <mesh filename="package://jsk_2014_picking_challenge/config/mesh/light/jigu_long2_left_kari2.dae" scale="0.001 0.001 0.001"/>
       </geometry>
       <material name="white">
@@ -68,20 +67,5 @@
     <collision>
       <geometry>
-        <cylinder radius="${width}" length="${bodylen_side2}"/>
-      </geometry>
-    </collision>
-  </link>
-  <link name="custom_vacuum_link_side2_base">
-    <visual>
-      <geometry>
-        <cylinder radius="${width_side2_base}" length="${bodylen_side2_base}"/>
-      </geometry>
-      <material name="white">
-        <color rgba="1 1 1 1"/>
-      </material>
-    </visual>
-    <collision>
-      <geometry>
-        <box size="0.001 0.001 0.001" />
+        <cylinder radius="${width_base}" length="${bodylen_base}"/>
       </geometry>
     </collision>
@@ -89,26 +73,21 @@
   <joint name="right_custom_joint" type="fixed">
     <parent link="right_wrist"/>
-    <child link="custom_vacuum_link"/>
+    <child link="right_custom_vacuum_link"/>
     <origin rpy="0 0 0" xyz="${right_wrist_offset_x} 0 0.18" />
   </joint>
   <joint name="right_custom_joint_base" type="fixed">
     <parent link="right_wrist"/>
-    <child link="custom_vacuum_link_base"/>
-    <origin rpy="0 0 0" xyz="${right_wrist_offset_x} 0 0.11" />
+    <child link="right_custom_vacuum_link_base"/>
+    <origin rpy="0 0 1.57" xyz="${right_wrist_offset_x} 0 0.11" />
   </joint>
-  <joint name="right_custom_joint_side" type="fixed">
-    <parent link="right_wrist"/>
-    <child link="custom_vacuum_link_side"/>
-    <origin rpy="1.57 0 0" xyz="${right_wrist_offset_x} 0 0.15" />
+  <joint name="left_custom_joint" type="fixed">
+    <parent link="left_wrist"/>
+    <child link="left_custom_vacuum_link"/>
+    <origin rpy="0 0 0" xyz="${left_wrist_offset_x} 0 0.18" />
   </joint>
-  <joint name="right_custom_joint_side2" type="fixed">
-    <parent link="right_wrist"/>
-    <child link="custom_vacuum_link_side2"/>
-    <origin rpy="0 0 0" xyz="${right_wrist_offset_x} 0 0.08" />
-  </joint>
-  <joint name="right_custom_joint_side2_base" type="fixed">
-    <parent link="right_wrist"/>
-    <child link="custom_vacuum_link_side2_base"/>
-    <origin rpy="0 0 0" xyz="${right_wrist_offset_x} 0 0.04" />
+  <joint name="left_custom_joint_base" type="fixed">
+    <parent link="left_wrist"/>
+    <child link="left_custom_vacuum_link_base"/>
+    <origin rpy="0 0 1.57" xyz="${left_wrist_offset_x} 0 0.11" />
   </joint>
 </robot>

Commit message: [baxter_white_hand_urdf.xacro] Update colision for vacuum pipe

File: jsk_2015_05_baxter_apc/config/baxter_white_hand.urdf.xacro (robot description, xacro)
@@ -3,8 +3,8 @@
   <xacro:include filename="$(find baxter_description)/urdf/baxter_simple.urdf" />
   <xacro:property name="width" value=".02" />
-  <xacro:property name="width_base" value=".04" />
+  <xacro:property name="width_base" value=".1" />
   <xacro:property name="width_side2_base" value=".035" />
   <xacro:property name="bodylen" value=".49" />
-  <xacro:property name="bodylen_base" value=".01" />
+  <xacro:property name="bodylen_base" value=".12" />
   <xacro:property name="right_wrist_offset_x" value="-0.01" />
   <xacro:property name="left_wrist_offset_x" value="-0.01" />
@@ -79,5 +79,5 @@
     <parent link="right_wrist"/>
     <child link="right_custom_vacuum_link_base"/>
-    <origin rpy="0 0 1.57" xyz="${right_wrist_offset_x} 0 0.11" />
+    <origin rpy="0 0 1.57" xyz="${right_wrist_offset_x} 0 0.08" />
   </joint>
   <joint name="left_custom_joint" type="fixed">
@@ -89,5 +89,5 @@
     <parent link="left_wrist"/>
     <child link="left_custom_vacuum_link_base"/>
-    <origin rpy="0 0 1.57" xyz="${left_wrist_offset_x} 0 0.11" />
+    <origin rpy="0 0 1.57" xyz="${left_wrist_offset_x} 0 0.08" />
   </joint>
 </robot>

Commit message: update baxter white hand xacro

File: jsk_2015_05_baxter_apc/config/baxter_white_hand.urdf.xacro (robot description, xacro)
@@ -74,20 +74,20 @@
     <parent link="right_wrist"/>
     <child link="right_custom_vacuum_link"/>
-    <origin rpy="0 0 0" xyz="${right_wrist_offset_x} 0 0.18" />
+    <origin rpy="0 0 0" xyz="${right_wrist_offset_x} 0.015 0.19" />
   </joint>
   <joint name="right_custom_joint_base" type="fixed">
     <parent link="right_wrist"/>
     <child link="right_custom_vacuum_link_base"/>
-    <origin rpy="0 0 1.57" xyz="${right_wrist_offset_x} 0 0.08" />
+    <origin rpy="0 0 1.57" xyz="${right_wrist_offset_x} 0.015 0.13" />
   </joint>
   <joint name="left_custom_joint" type="fixed">
     <parent link="left_wrist"/>
     <child link="left_custom_vacuum_link"/>
-    <origin rpy="0 0 0" xyz="${left_wrist_offset_x} 0 0.18" />
+    <origin rpy="0 0 0" xyz="${left_wrist_offset_x} -0.015 0.19" />
   </joint>
   <joint name="left_custom_joint_base" type="fixed">
     <parent link="left_wrist"/>
     <child link="left_custom_vacuum_link_base"/>
-    <origin rpy="0 0 1.57" xyz="${left_wrist_offset_x} 0 0.08" />
+    <origin rpy="0 0 1.57" xyz="${left_wrist_offset_x} -0.015 0.13" />
   </joint>
 </robot>

Commit message: Adjust kinect2 tf and baxter custom link after calibration of kinect2

File: jsk_2015_05_baxter_apc/config/baxter_white_hand.urdf.xacro (robot description, xacro)
@@ -74,20 +74,20 @@
     <parent link="right_wrist"/>
     <child link="right_custom_vacuum_link"/>
-    <origin rpy="0 0 0" xyz="${right_wrist_offset_x} 0.015 0.19" />
+    <origin rpy="0 0 0" xyz="${right_wrist_offset_x} 0 0.19" />
   </joint>
   <joint name="right_custom_joint_base" type="fixed">
     <parent link="right_wrist"/>
     <child link="right_custom_vacuum_link_base"/>
-    <origin rpy="0 0 1.57" xyz="${right_wrist_offset_x} 0.015 0.13" />
+    <origin rpy="0 0 1.57" xyz="${right_wrist_offset_x} -0 0.13" />
   </joint>
   <joint name="left_custom_joint" type="fixed">
     <parent link="left_wrist"/>
     <child link="left_custom_vacuum_link"/>
-    <origin rpy="0 0 0" xyz="${left_wrist_offset_x} -0.015 0.19" />
+    <origin rpy="0 0 0" xyz="${left_wrist_offset_x} 0 0.19" />
   </joint>
   <joint name="left_custom_joint_base" type="fixed">
     <parent link="left_wrist"/>
     <child link="left_custom_vacuum_link_base"/>
-    <origin rpy="0 0 1.57" xyz="${left_wrist_offset_x} -0.015 0.13" />
+    <origin rpy="0 0 1.57" xyz="${left_wrist_offset_x} -0 0.13" />
   </joint>
 </robot>

Commit message: Replace package name: jsk_2014_baxter_apc -> jsk_2015_05_baxter_apc

File: jsk_2015_05_baxter_apc/config/baxter_white_hand.urdf.xacro (robot description, xacro)
@@ -13,5 +13,5 @@
       <origin rpy="0 0 1.57" xyz="0 0 -0.07"/>
       <geometry>
-        <mesh filename="package://jsk_2014_baxter_apc/config/mesh/long1_simple.dae" scale="0.001 0.001 0.001"/>
+        <mesh filename="package://jsk_2015_05_baxter_apc/config/mesh/long1_simple.dae" scale="0.001 0.001 0.001"/>
       </geometry>
       <material name="white">
@@ -28,5 +28,5 @@
     <visual>
       <geometry>
-        <mesh filename="package://jsk_2014_baxter_apc/config/mesh/light/jigu_long2_right_kari1.dae" scale="0.001 0.001 0.001"/>
+        <mesh filename="package://jsk_2015_05_baxter_apc/config/mesh/light/jigu_long2_right_kari1.dae" scale="0.001 0.001 0.001"/>
       </geometry>
       <material name="white">
@@ -44,5 +44,5 @@
       <origin rpy="0 0 1.57" xyz="0 0 -0.07"/>
       <geometry>
-        <mesh filename="package://jsk_2014_baxter_apc/config/mesh/long1_simple.dae" scale="0.001 0.001 0.001"/>
+        <mesh filename="package://jsk_2015_05_baxter_apc/config/mesh/long1_simple.dae" scale="0.001 0.001 0.001"/>
       </geometry>
       <material name="white">
@@ -59,5 +59,5 @@
     <visual>
       <geometry>
-        <mesh filename="package://jsk_2014_baxter_apc/config/mesh/light/jigu_long2_left_kari2.dae" scale="0.001 0.001 0.001"/>
+        <mesh filename="package://jsk_2015_05_baxter_apc/config/mesh/light/jigu_long2_left_kari2.dae" scale="0.001 0.001 0.001"/>
       </geometry>
       <material name="white">
