Commit message: add baxter white hand dae model

File: jsk_2015_05_baxter_apc/config/baxter_white_hand.urdf (robot description, URDF)
Before this commit: robot baxter_custom_white, 54 links, 53 joints
Links:
- link custom_vacuum_link: geometry collision cylinder length=0.14 radius=0.02; visual mesh filename=package://jsk_2014_picking_challenge/config/mesh/jigukai13.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

File: jsk_2015_05_baxter_apc/config/baxter_white_hand.urdf.xacro (robot description, xacro)
@@ -13,5 +13,5 @@
     <visual>
       <geometry>
-        <cylinder radius="${width}" length="${bodylen}"/>
+        <mesh filename="package://jsk_2014_picking_challenge/config/mesh/jigukai13.dae"/>
       </geometry>
       <material name="white">

Commit message: update model rotation and pos

File: jsk_2015_05_baxter_apc/config/baxter_white_hand.urdf (robot description, URDF)
Before this commit: robot baxter_custom_white, 54 links, 53 joints
Links:
- link custom_vacuum_link_base: geometry collision cylinder length=0.01 radius=0.04; visual cylinder length=0 radius=0
- link custom_vacuum_link_side: geometry collision cylinder length=0.15 radius=0.02; visual cylinder length=0 radius=0
- link custom_vacuum_link_side2: geometry collision cylinder length=0.12 radius=0.02; visual cylinder length=0 radius=0
- link custom_vacuum_link_side2_base: geometry collision cylinder length=0 radius=0; visual cylinder length=0.06 radius=0.035

File: jsk_2015_05_baxter_apc/config/baxter_white_hand.urdf.xacro (robot description, xacro)
@@ -12,4 +12,5 @@
   <link name="custom_vacuum_link">
     <visual>
+      <origin rpy="0 0 1.57" xyz="0 0 -0.07"/>
       <geometry>
         <mesh filename="package://jsk_2014_picking_challenge/config/mesh/jigukai13.dae"/>
@@ -28,5 +29,5 @@
     <visual>
       <geometry>
-        <cylinder radius="${width_base}" length="${bodylen_base}"/>
+        <cylinder radius="0" length="0"/>
       </geometry>
       <material name="white">
@@ -43,5 +44,5 @@
     <visual>
       <geometry>
-        <cylinder radius="${width}" length="${bodylen_side}"/>
+        <cylinder radius="0" length="0"/>
       </geometry>
       <material name="white">
@@ -58,5 +59,5 @@
     <visual>
       <geometry>
-        <cylinder radius="${width}" length="${bodylen_side2}"/>
+        <cylinder radius="0" length="0"/>
       </geometry>
       <material name="white">
@@ -81,5 +82,5 @@
     <collision>
       <geometry>
-        <cylinder radius="${width_side2_base}" length="${bodylen_side2_base}"/>
+        <cylinder radius="0" length="0"/>
       </geometry>
     </collision>

Commit message: Add new baxter long vacuum DAE

File: jsk_2015_05_baxter_apc/config/baxter_white_hand.urdf (robot description, URDF)
Before this commit: robot baxter_custom_white, 54 links, 53 joints
Links:
- link custom_vacuum_link: geometry collision cylinder length=0.14 radius=0.02; visual mesh filename=package://jsk_2014_picking_challenge/config/mesh/long1.dae scale=0.001 0.001 0.001
- link custom_vacuum_link_base: geometry collision cylinder length=0.01 radius=0.04; visual mesh filename=package://jsk_2014_picking_challenge/config/mesh/jigukailon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 scale=0.001 0.001 0.001
Joints:
- joint right_custom_joint_base: origin xyz=0 0 0.11 rpy=0 0 0 -> xyz=0 0 0.11 rpy=0 0 1.57

File: jsk_2015_05_baxter_apc/config/baxter_white_hand.urdf.xacro (robot description, xacro)
@@ -14,5 +14,5 @@
       <origin rpy="0 0 1.57" xyz="0 0 -0.07"/>
       <geometry>
-        <mesh filename="package://jsk_2014_picking_challenge/config/mesh/jigukai13.dae"/>
+        <mesh filename="package://jsk_2014_picking_challenge/config/mesh/long1.dae" scale="0.001 0.001 0.001"/>
       </geometry>
       <material name="white">
@@ -29,5 +29,5 @@
     <visual>
       <geometry>
-        <cylinder radius="0" length="0"/>
+        <mesh filename="package://jsk_2014_picking_challenge/config/mesh/jigukailong2.dae" scale="0.001 0.001 0.001"/>
       </geometry>
       <material name="white">
@@ -94,5 +94,5 @@
     <parent link="right_wrist"/>
     <child link="custom_vacuum_link_base"/>
-    <origin rpy="0 0 0" xyz="0 0 0.11" />
+    <origin rpy="0 0 1.57" xyz="0 0 0.11" />
   </joint>
   <joint name="right_custom_joint_side" type="fixed">

Commit message: publish /gripper_grabbed/limb/left/state2, checking wrench forces

File: jsk_2015_05_baxter_apc/config/baxter_white_hand.urdf (robot description, URDF)
Before this commit: robot baxter_custom_white, 54 links, 53 joints
Links:
- link custom_vacuum_link: geometry collision cylinder length=0.45 radius=0.02; visual mesh filename=package://jsk_2014_picking_challenge/config/mesh/long1_simp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 scale=0.001 0.001 0.001
- link custom_vacuum_link_side: geometry collision cylinder length=0.15 radius=0.02; visual box size=0.001 0.001 0.001
- link custom_vacuum_link_side2: geometry collision cylinder length=0.12 radius=0.02; visual box size=0.001 0.001 0.001
- link custom_vacuum_link_side2_base: geometry collision box size=0.001 0.001 0.001; visual cylinder length=0.06 radius=0.035
- link head: geometry collision sphere radius=0.001; visual mesh filename=package://baxter_description/meshes/head/H0_simple.STL
- link left_lower_elbow: geometry collision cylinder length=0.10 radius=0.06; visual mesh filename=package://baxter_description/meshes/lower_elbow/E1_simple.S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
- link left_lower_forearm: geometry collision cylinder length=0.10 radius=0.06; visual mesh filename=package://baxter_description/meshes/lower_forearm/W1_simple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
- link left_lower_shoulder: geometry collision cylinder length=0.12 radius=0.06; visual mesh filename=package://baxter_description/meshes/lower_shoulder/S1_simpl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
- link left_upper_elbow: geometry collision cylinder length=0.107 radius=0.06; visual mesh filename=package://baxter_description/meshes/upper_elbow/E0_simple.S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
- link left_upper_forearm: geometry collision cylinder length=0.088 radius=0.06; visual mesh filename=package://baxter_description/meshes/upper_forearm/W0_simple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
- link left_upper_shoulder: geometry collision cylinder length=0.2722 radius=0.06; visual mesh filename=package://baxter_description/meshes/upper_shoulder/S0_simpl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
- link left_wrist: geometry collision cylinder length=0.165 radius=0.06; visual mesh filename=package://baxter_description/meshes/wrist/W2_simple.STL
- link pedestal: geometry collision mesh filename=package://baxter_description/meshes/base/pedestal_link_coll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; visual mesh filename=package://baxter_description/meshes/base/pedestal_link_coll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
- link right_lower_elbow: geometry collision cylinder length=0.10 radius=0.06; visual mesh filename=package://baxter_description/meshes/lower_elbow/E1_simple.S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
- link right_lower_forearm: geometry collision cylinder length=0.10 radius=0.06; visual mesh filename=package://baxter_description/meshes/lower_forearm/W1_simple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
- link right_lower_shoulder: geometry collision cylinder length=0.12 radius=0.06; visual mesh filename=package://baxter_description/meshes/lower_shoulder/S1_simpl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
- link right_upper_elbow: geometry collision cylinder length=0.107 radius=0.06; visual mesh filename=package://baxter_description/meshes/upper_elbow/E0_simple.S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
- link right_upper_forearm: geometry collision cylinder length=0.088 radius=0.06; visual mesh filename=package://baxter_description/meshes/upper_forearm/W0_simple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
- link right_upper_shoulder: geometry collision cylinder length=0.2722 radius=0.06; visual mesh filename=package://baxter_description/meshes/upper_shoulder/S0_simpl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
- link right_wrist: geometry collision cylinder length=0.165 radius=0.06; visual mesh filename=package://baxter_description/meshes/wrist/W2_simple.STL
- link screen: geometry collision sphere radius=0.001; visual mesh filename=package://baxter_description/meshes/head/H1_simple.STL
- link torso: geometry collision mesh filename=package://baxter_description/meshes/torso/base_link_collisi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; visual mesh filename=package://baxter_description/meshes/torso/base_link_collisi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
Joints:
- joint right_custom_joint: origin xyz=0 0 0.18 rpy=0 0 0 -> xyz=-0.04 0 0.18 rpy=0 0 0
- joint right_custom_joint_base: origin xyz=0 0 0.11 rpy=0 0 1.57 -> xyz=-0.04 0 0.11 rpy=0 0 0
- joint right_custom_joint_side: origin xyz=0 0.05 0.15 rpy=1.57 0 0 -> xyz=-0.04 0 0.15 rpy=1.57 0 0
- joint right_custom_joint_side2: origin xyz=0 0.1 0.08 rpy=0 0 0 -> xyz=-0.04 0 0.08 rpy=0 0 0
- joint right_custom_joint_side2_base: origin xyz=0 0.1 0.04 rpy=0 0 0 -> xyz=-0.04 0 0.04 rpy=0 0 0

Commit message: Rename pkg: jsk_2014_picking_challenge -> jsk_2015_05_baxter_apc

File: jsk_2015_05_baxter_apc/config/baxter_white_hand.urdf (robot description, URDF)
Before this commit: robot baxter, 54 links, 53 joints
Links:
- link custom_vacuum_link: geometry collision cylinder length=0.45 radius=0.02; visual mesh filename=package://jsk_2015_05_baxter_apc/config/mesh/long1_simple.d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 scale=0.001 0.001 0.001
- link custom_vacuum_link_base: geometry collision cylinder length=0.01 radius=0.04; visual mesh filename=package://jsk_2015_05_baxter_apc/config/mesh/jigukailong2_s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 scale=0.001 0.001 0.001

File: jsk_2015_05_baxter_apc/config/baxter_white_hand.urdf.xacro (robot description, xacro)
@@ -13,5 +13,5 @@
       <origin rpy="0 0 1.57" xyz="0 0 -0.07"/>
       <geometry>
-        <mesh filename="package://jsk_2014_picking_challenge/config/mesh/long1_simple.dae" scale="0.001 0.001 0.001"/>
+        <mesh filename="package://jsk_2015_05_baxter_apc/config/mesh/long1_simple.dae" scale="0.001 0.001 0.001"/>
       </geometry>
       <material name="white">
@@ -28,5 +28,5 @@
     <visual>
       <geometry>
-        <mesh filename="package://jsk_2014_picking_challenge/config/mesh/light/jigu_long2_right_kari1.dae" scale="0.001 0.001 0.001"/>
+        <mesh filename="package://jsk_2015_05_baxter_apc/config/mesh/light/jigu_long2_right_kari1.dae" scale="0.001 0.001 0.001"/>
       </geometry>
       <material name="white">
@@ -44,5 +44,5 @@
       <origin rpy="0 0 1.57" xyz="0 0 -0.07"/>
       <geometry>
-        <mesh filename="package://jsk_2014_picking_challenge/config/mesh/long1_simple.dae" scale="0.001 0.001 0.001"/>
+        <mesh filename="package://jsk_2015_05_baxter_apc/config/mesh/long1_simple.dae" scale="0.001 0.001 0.001"/>
       </geometry>
       <material name="white">
@@ -59,5 +59,5 @@
     <visual>
       <geometry>
-        <mesh filename="package://jsk_2014_picking_challenge/config/mesh/light/jigu_long2_left_kari2.dae" scale="0.001 0.001 0.001"/>
+        <mesh filename="package://jsk_2015_05_baxter_apc/config/mesh/light/jigu_long2_left_kari2.dae" scale="0.001 0.001 0.001"/>
       </geometry>
       <material name="white">
