Commit message: [jsk_2015_apc_common] Move kiva_pod model files to urdf/ & meshes/

File: jsk_apc2015_common/urdf/pod_lowres.urdf (robot description, URDF)
Before this commit: robot kiva_pod, 1 links, 0 joints
Links:
- link kiva_pod_body: geometry collision mesh filename=package://jsk_2015_apc_common/meshes/pod_lowres/pod_lowres.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; visual mesh filename=package://jsk_2015_apc_common/meshes/pod_lowres/pod_lowres.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
