Commit message: Revert "[jsk_2015_apc_common] Move kiva_pod model files to urdf/ & meshes/"
This reverts commit 91a818229d2b6e9faa66912bbbef7370941d30f5.

File: jsk_apc2015_common/kiva_pod/urdf/kiva_pod.urdf (robot description, URDF)
Before this commit: robot kiva_pod, 1 links, 0 joints
Links:
- link kiva_pod_body: geometry collision mesh filename=package://jsk_2015_apc_common/kiva_pod/meshes/pod_lowres.stl; visual mesh filename=package://jsk_2015_apc_common/kiva_pod/meshes/pod_lowres.stl
