Commit message: [jsk_2015_05_baxter_apc] Move meshes location

File: jsk_2015_05_baxter_apc/urdf/baxter_custom.xacro (robot description, xacro)
@@ -13,5 +13,5 @@
       <origin rpy="0 0 1.57" xyz="0 0 -0.07"/>
       <geometry>
-        <mesh filename="package://jsk_2015_05_baxter_apc/config/mesh/long1_simple.dae" scale="0.001 0.001 0.001"/>
+        <mesh filename="package://jsk_2015_05_baxter_apc/meshes/long1_simple.dae" scale="0.001 0.001 0.001"/>
       </geometry>
       <material name="white">
@@ -28,5 +28,5 @@
     <visual>
       <geometry>
-        <mesh filename="package://jsk_2015_05_baxter_apc/config/mesh/light/jigu_long2_right_kari1.dae" scale="0.001 0.001 0.001"/>
+        <mesh filename="package://jsk_2015_05_baxter_apc/meshes/light/jigu_long2_right_kari1.dae" scale="0.001 0.001 0.001"/>
       </geometry>
       <material name="white">
@@ -44,5 +44,5 @@
       <origin rpy="0 0 1.57" xyz="0 0 -0.07"/>
       <geometry>
-        <mesh filename="package://jsk_2015_05_baxter_apc/config/mesh/long1_simple.dae" scale="0.001 0.001 0.001"/>
+        <mesh filename="package://jsk_2015_05_baxter_apc/meshes/long1_simple.dae" scale="0.001 0.001 0.001"/>
       </geometry>
       <material name="white">
@@ -59,5 +59,5 @@
     <visual>
       <geometry>
-        <mesh filename="package://jsk_2015_05_baxter_apc/config/mesh/light/jigu_long2_left_kari2.dae" scale="0.001 0.001 0.001"/>
+        <mesh filename="package://jsk_2015_05_baxter_apc/meshes/light/jigu_long2_left_kari2.dae" scale="0.001 0.001 0.001"/>
       </geometry>
       <material name="white">
