Commit message: [jsk_2015_apc_common] Adjust kiva pod

File: jsk_apc2015_common/models/kiva_pod/urdf/pod_lowres_convex.xacro (robot description, xacro)
@@ -117,10 +117,10 @@
   <link name="kiva_pod_y_part1">
     <visual>
-      <origin rpy="0 0 0" xyz="0 0.15 0"/>
+      <origin rpy="0 0 0" xyz="0 0.16 0"/>
       <geometry><box size="${y_part_size}"/></geometry>
       <material name="darkgray"><color rgba=".2 .2 .2 1"/></material>
     </visual>
     <collision>
-      <origin rpy="0 0 0" xyz="0 0.15 0"/>
+      <origin rpy="0 0 0" xyz="0 0.16 0"/>
       <geometry><box size="${y_part_size}"/></geometry>
     </collision>
@@ -132,10 +132,10 @@
   <link name="kiva_pod_y_part2">
     <visual>
-      <origin rpy="0 0 0" xyz="0 -.15 0"/>
+      <origin rpy="0 0 0" xyz="0 -.16 0"/>
       <geometry><box size="${y_part_size}"/></geometry>
       <material name="darkgray"><color rgba=".2 .2 .2 1"/></material>
     </visual>
     <collision>
-      <origin rpy="0 0 0" xyz="0 -.15 0"/>
+      <origin rpy="0 0 0" xyz="0 -.16 0"/>
       <geometry><box size="${y_part_size}"/></geometry>
     </collision>
