Commit message: [jsk_2015_apc_common] kiva_pod -> models/kiva_pod

File: jsk_apc2015_common/models/kiva_pod/urdf/pod_lowres.urdf (robot description, URDF)
Before this commit: robot kiva_pod, 1 links, 0 joints
Links:
- link kiva_pod_body: geometry collision mesh filename=package://jsk_2015_apc_common/models/kiva_pod/meshes/pod_lo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; visual mesh filename=package://jsk_2015_apc_common/models/kiva_pod/meshes/pod_lo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

Commit message: jsk_2015_apc_common -> jsk_apc2015_common

File: jsk_apc2015_common/models/kiva_pod/urdf/pod_lowres.urdf (robot description, URDF)
Before this commit: robot kiva_pod, 1 links, 0 joints
Links:
- link kiva_pod_body: geometry collision mesh filename=package://jsk_apc2015_common/models/kiva_pod/meshes/pod_low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; visual mesh filename=package://jsk_apc2015_common/models/kiva_pod/meshes/pod_low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
