Commit message: Fix collision of apc_order_bin model

File: jsk_apc2015_common/models/apc_order_bin/urdf/order_bin.urdf (robot description, URDF)
Before this commit: robot order_bin, 5 links, 4 joints
Links:
- link order_bin_base: geometry collision box size=0.35 0.53 .03; visual box size=0.35 0.53 .03

File: jsk_apc2015_common/models/apc_order_bin/urdf/order_bin.xacro (robot description, xacro)
@@ -12,11 +12,11 @@
   <link name="order_bin_base">
     <visual>
-      <origin rpy="0 0 0" xyz="0 0 .015"/>
+      <origin rpy="0 0 0" xyz="0 0 0"/>
       <geometry><box size="${z_part_size}"/></geometry>
       <material name="red" />
     </visual>
     <collision>
-      <origin rpy="0 0 0" xyz="0 0 ${z_size/2}"/>
-      <geometry><box size="${x_part_size}"/></geometry>
+      <origin rpy="0 0 0" xyz="0 0 0"/>
+      <geometry><box size="${z_part_size}"/></geometry>
       <material name="red" />
     </collision>
