Commit message: add softkinetic xacro

File: jsk_2016_01_baxter_apc/robots/baxter.xacro (robot description, xacro)
@@ -1,10 +1,8 @@
 <?xml version="1.0"?>
-<robot xmlns:xacro="http://ros.org/wiki/xacro" name="baxter_creative">
-  <xacro:include filename="$(find jsk_2015_05_baxter_apc)/robots/baxter.xacro"/>
-  <!-- Creative Camera -->
-  <xacro:include filename="$(find softkinetic_camera)/urdf/senz3d.urdf.xacro"/>
-  <xacro:sensor_senz3d name="left_softkinetic_camera" parent="left_wrist">
-    <origin rpy="0 -${M_PI/2} ${M_PI}" xyz="-0.048 0.0 0.10"/>
-  </xacro:sensor_senz3d>
+<robot xmlns:xacro="http://ros.org/wiki/xacro" name="baxter">
+  <xacro:include filename="$(find jsk_2015_05_baxter_apc)/robots/baxter.xacro" />
+  <!-- Arm Camera -->
+  <xacro:include filename="$(find jsk_2016_01_baxter_apc)/robots/right_arm_camera.xacro"/>
+  <xacro:include filename="$(find jsk_2016_01_baxter_apc)/robots/left_arm_camera.xacro"/>
   <!-- Vaccum Gripper-->
   <xacro:include filename="$(find jsk_2016_01_baxter_apc)/robots/left_vaccum_gripper.xacro"/>
