Commit message: fix softkinetic position

File: jsk_2016_01_baxter_apc/robots/left_arm_camera.xacro (robot description, xacro)
@@ -2,6 +2,6 @@
 <robot xmlns:xacro="http://ros.org/wiki/xacro" name="left_arm_camera">
   <xacro:include filename="$(find jsk_2016_01_baxter_apc)/robots/softkinetic_camera/senz3d.urdf.xacro"/>
-  <xacro:sensor_senz3d name="left_softkinetic_camera" parent="left_wrist">
-    <origin rpy="0 -${M_PI/2} ${M_PI}" xyz="-0.048 0.0 0.10"/>
+  <xacro:sensor_senz3d name="left_softkinetic_camera" parent="left_hand">
+    <origin rpy="0 -${M_PI/2} ${M_PI}" xyz="-0.060 0.022 0"/>
   </xacro:sensor_senz3d>
 </robot>

File: jsk_2016_01_baxter_apc/robots/right_arm_camera.xacro (robot description, xacro)
@@ -2,6 +2,6 @@
 <robot xmlns:xacro="http://ros.org/wiki/xacro" name="right_arm_camera">
   <xacro:include filename="$(find jsk_2016_01_baxter_apc)/robots/softkinetic_camera/senz3d.urdf.xacro"/>
-  <xacro:sensor_senz3d name="right_softkinetic_camera" parent="right_wrist">
-    <origin rpy="0 -${M_PI/2} ${M_PI}" xyz="-0.048 0.0 0.10"/>
+  <xacro:sensor_senz3d name="right_softkinetic_camera" parent="right_hand">
+    <origin rpy="0 -${M_PI/2} ${M_PI}" xyz="-0.060 0.022 0"/>
   </xacro:sensor_senz3d>
 </robot>

Commit message: fix position of softkinetic_camera

File: jsk_2016_01_baxter_apc/robots/left_arm_camera.xacro (robot description, xacro)
@@ -3,5 +3,5 @@
   <xacro:include filename="$(find jsk_2016_01_baxter_apc)/robots/softkinetic_camera/senz3d.urdf.xacro"/>
   <xacro:sensor_senz3d name="left_softkinetic_camera" parent="left_hand">
-    <origin rpy="0 -${M_PI/2} ${M_PI}" xyz="-0.060 0.022 0"/>
+    <origin rpy="0 -${M_PI/2} ${M_PI}" xyz="-0.048 0 0.025"/>
   </xacro:sensor_senz3d>
 </robot>

File: jsk_2016_01_baxter_apc/robots/right_arm_camera.xacro (robot description, xacro)
@@ -3,5 +3,5 @@
   <xacro:include filename="$(find jsk_2016_01_baxter_apc)/robots/softkinetic_camera/senz3d.urdf.xacro"/>
   <xacro:sensor_senz3d name="right_softkinetic_camera" parent="right_hand">
-    <origin rpy="0 -${M_PI/2} ${M_PI}" xyz="-0.060 0.022 0"/>
+    <origin rpy="0 -${M_PI/2} ${M_PI}" xyz="-0.048 0 0.025"/>
   </xacro:sensor_senz3d>
 </robot>
