Commit message: Add gripper-v5 visual to right hand

File: jsk_2016_01_baxter_apc/robots/right_vacuum_gripper.xacro (robot description, xacro)
@@ -3,129 +3,151 @@
   <xacro:include filename="$(find jsk_2016_01_baxter_apc)/robots/common_constants.xacro"/>
   <!--Link bodies-->
-  <xacro:property name="rect_tube_l" value="0.285" />
-  <xacro:property name="rect_tube_h" value="0.06" />
-  <xacro:property name="rect_tube_w" value="0.0952" />
-  <xacro:property name="cyl_tube_x" value="0.005" />
-  <xacro:property name="cyl_tube_z" value="0.038" />
-  <xacro:property name="cyl_tube_r" value="0.018" />
-  <xacro:property name="cyl_tube_l" value="0.107" />
-  <xacro:property name="connection_z" value="-0.00725" />
-  <xacro:property name="connection_r" value="0.03" />
-  <xacro:property name="connection_l" value="0.0905" />
-  <xacro:property name="pad_base_z" value="0.025" />
-  <xacro:property name="pad_base_w" value="0.09" />
-  <xacro:property name="pad_base_h" value="0.038" />
-  <xacro:property name="pad_base_d" value="0.06" />
-  <xacro:property name="pad_r" value="0.026" />
-  <xacro:property name="pad_l" value="0.03" />
-  <xacro:property name="pad_x" value="-0.0005" />
-  <xacro:property name="pad_y" value="0.0085" />
-  <xacro:property name="pad_z" value="0.07" />
+  <xacro:property name="pad_with_base_offset_x" value="-0.048" />
+  <xacro:property name="pad_with_base_offset_y" value="-0.0005" />
+  <xacro:property name="pad_with_base_offset_z" value="-0.302" />
   <!--Joints-->
-  <xacro:property name="right_hand_offset_x" value="-0.01" />
-  <xacro:property name="right_hand_offset_z" value="0" />
-  <xacro:property name="right_gripper_joint_offset_x" value="0.005" />
-  <xacro:property name="right_gripper_joint_offset_y" value="-0.0085" />
-  <xacro:property name="right_gripper_joint_offset_z" value="0.264" />
+  <xacro:property name="hand_offset_x" value="-0.01" />
+  <xacro:property name="hand_offset_z" value="0" />
+  <xacro:property name="pad_joint_offset_x" value="0.048" />
+  <xacro:property name="pad_joint_offset_y" value="0.0005" />
+  <xacro:property name="pad_joint_offset_z" value="0.302" />
+  <xacro:property name="finger_base_offset_z" value="0.291352" />
+  <xacro:property name="finger_base_offset_x" value="-0.014" />
+  <xacro:property name="l_finger_base_offset_y" value="0.026" />
+  <xacro:property name="r_finger_base_offset_y" value="-0.026" />
+  <!--Link bodies-->
   <link name="right_gripper_base">
     <visual>
-      <origin rpy="${M_PI/2} 0 -${M_PI/2}" xyz="0 0 0"/>
+      <origin rpy="${M_PI/2} 0 ${M_PI/2}" xyz="0 0 0"/>
       <geometry>
         <mesh filename="package://jsk_2016_01_baxter_apc/meshes/visual/right_gripper_base.stl" scale="0.001 0.001 0.001"/>
       </geometry>
-      <material name="white">
-        <color rgba="1 1 1 1"/>
-      </material>
-    </visual>
-    <!--When using this stl file, robot_self_filter doesn't work-->
-    <!--<collision>
-      <origin rpy="${M_PI/2} 0 -${M_PI/2}" xyz="0 0 0"/>
-      <geometry>
-        <mesh filename="package://jsk_2016_01_baxter_apc/meshes/collision/right_gripper_base.stl" scale="0.001 0.001 0.001"/>
-      </geometry>
-    </collision>-->
-    <collision>
-      <origin rpy="0 0 0" xyz="0 0 ${rect_tube_l/2}"/>
-      <geometry>
-        <box size="${rect_tube_h} ${rect_tube_w} ${rect_tube_l}"/>
-      </geometry>
-    </collision>
-    <collision>
-      <origin rpy="${M_PI/2} 0 0" xyz="${cyl_tube_x} -${cyl_tube_l/2} ${cyl_tube_z}"/>
-      <geometry>
-        <cylinder radius="${cyl_tube_r}" length="${cyl_tube_l}"/>
-      </geometry>
-    </collision>
-    <collision>
-      <origin rpy="0 0 0" xyz="${cyl_tube_x} -${cyl_tube_l} ${connection_z}"/>
-      <geometry>
-        <cylinder radius="${connection_r}" length="${connection_l}"/>
-      </geometry>
-    </collision>
-  </link>
-  <link name="right_gripper_vacuum_pad_base">
-    <visual>
-      <origin rpy="${M_PI/2} 0 -${M_PI/2}" xyz="0 0 0"/>
-      <geometry>
-        <mesh filename="package://jsk_2016_01_baxter_apc/meshes/visual/right_gripper_vacuum_pad_base.stl" scale="0.001 0.001 0.001"/>
-      </geometry>
-      <material name="gray">
+      <material name="lightgrey">
         <color rgba="0.5 0.5 0.5 1"/>
       </material>
     </visual>
-    <!--When using this stl file, robot_self_filter doesn't work-->
-    <!--<collision>
-      <origin rpy="${M_PI/2} 0 -${M_PI/2}" xyz="0 0 0"/>
+    <!--FIXME: Add collision-->
+  </link>
+  <link name="right_gripper_tube">
+    <visual>
+      <origin rpy="${M_PI/2} 0 ${M_PI/2}" xyz="0 0 0"/>
       <geometry>
-        <mesh filename="package://jsk_2016_01_baxter_apc/meshes/collision/right_gripper_vacuum_pad_base.stl" scale="0.001 0.001 0.001"/>
+        <mesh filename="package://jsk_2016_01_baxter_apc/meshes/visual/right_gripper_tube.stl" scale="0.001 0.001 0.001"/>
       </geometry>
-    </collision>-->
-    <collision>
-      <origin rpy="0 0 0" xyz="0 0 ${pad_base_z}"/>
-      <geometry>
-        <box size="${pad_base_h} ${pad_base_w} ${pad_base_d}"/>
-      </geometry>
-    </collision>
-  </link>
-  <link name="right_gripper_vacuum_pad">
-    <visual>
-      <origin rpy="${M_PI/2} 0 -${M_PI/2}" xyz="0 0 0"/>
-      <geometry>
-        <mesh filename="package://jsk_2016_01_baxter_apc/meshes/visual/right_gripper_vacuum_pad.stl" scale="0.001 0.001 0.001"/>
-      </geometry>
-      <material name="green">
-        <color rgba="0 1 0 1"/>
+      <material name="lightgrey">
+        <color rgba="0.5 0.5 0.5 1"/>
       </material>
     </visual>
-    <!--When using this stl file, robot_self_filter doesn't work-->
-    <!--<collision>
-      <origin rpy="${M_PI/2} 0 -${M_PI/2}" xyz="0 0 0"/>
+    <!--FIXME: Add collision-->
+  </link>
+  <link name="right_gripper_pad_with_base">
+    <visual>
+      <origin rpy="${M_PI/2} 0 ${M_PI/2}" xyz="${pad_with_base_offset_x} ${pad_with_base_offset_y} ${pad_with_base_offset_z}"/>
       <geometry>
-        <mesh filename="package://jsk_2016_01_baxter_apc/meshes/collision/right_gripper_vacuum_pad.stl" scale="0.001 0.001 0.001"/>
+        <mesh filename="package://jsk_2016_01_baxter_apc/meshes/visual/right_gripper_pad_with_base.stl" scale="0.001 0.001 0.001"/>
       </geometry>
-    </collision>-->
-    <collision>
-      <origin rpy="0 0 0" xyz="${pad_x} ${pad_y} ${pad_z}"/>
+      <material name="lightgrey">
+        <color rgba="0.5 0.5 0.5 1"/>
+      </material>
+    </visual>
+    <!--FIXME: Add collision-->
+  </link>
+  <link name="right_gripper_r_finger_base">
+    <visual>
+      <origin rpy="${M_PI/2} 0 ${M_PI}" xyz="0 0 0"/>
       <geometry>
-        <cylinder radius="${pad_r}" length="${pad_l}"/>
+        <mesh filename="package://jsk_2016_01_baxter_apc/meshes/visual/finger_base.stl" scale="0.001 0.001 0.001"/>
       </geometry>
-    </collision>
+      <material name="lightgrey">
+        <color rgba="0.5 0.5 0.5 1"/>
+      </material>
+    </visual>
+    <!--FIXME: Add collision-->
   </link>
+  <link name="right_gripper_l_finger_base">
+    <visual>
+      <origin rpy="${M_PI/2} 0 0" xyz="0 0 0"/>
+      <geometry>
+        <mesh filename="package://jsk_2016_01_baxter_apc/meshes/visual/finger_base.stl" scale="0.001 0.001 0.001"/>
+      </geometry>
+      <material name="lightgrey">
+        <color rgba="0.5 0.5 0.5 1"/>
+      </material>
+    </visual>
+    <!--FIXME: Add collision-->
+  </link>
+  <link name="right_gripper_r_finger">
+    <visual>
+      <origin rpy="${M_PI/2} 0 ${M_PI}" xyz="0 0 0"/>
+      <geometry>
+        <mesh filename="package://jsk_2016_01_baxter_apc/meshes/visual/finger.stl" scale="0.001 0.001 0.001"/>
+      </geometry>
+      <material name="lightgrey">
+        <color rgba="0.5 0.5 0.5 1"/>
+      </material>
+    </visual>
+    <!--FIXME: Add collision-->
+  </link>
+  <link name="right_gripper_l_finger">
+    <visual>
+      <origin rpy="${M_PI/2} 0 0" xyz="0 0 0"/>
+      <geometry>
+        <mesh filename="package://jsk_2016_01_baxter_apc/meshes/visual/finger.stl" scale="0.001 0.001 0.001"/>
+      </geometry>
+      <material name="lightgrey">
+        <color rgba="0.5 0.5 0.5 1"/>
+      </material>
+    </visual>
+    <!--FIXME: Add collision-->
+  </link>
+  <!--Joints-->
   <joint name="right_gripper_base_fixed" type="fixed">
-    <origin rpy="0 0 0" xyz="${right_hand_offset_x} 0 ${right_hand_offset_z}" />
+    <origin rpy="0 0 0" xyz="${hand_offset_x} 0 ${hand_offset_z}" />
     <parent link="right_hand"/>
     <child link="right_gripper_base"/>
   </joint>
+  <joint name="right_gripper_prismatic_joint" type="prismatic">
+    <origin rpy="0 0 0" xyz="0 0 0" />
+    <parent link="right_gripper_base"/>
+    <child link="right_gripper_tube"/>
+    <axis xyz="0 0 1"/>
+    <limit lower="0" upper="0.124" effort="0" velocity="0.024"/>
+  </joint>
   <joint name="right_gripper_vacuum_pad_joint" type="revolute">
-    <origin rpy="0 0 0" xyz="${right_gripper_joint_offset_x} ${right_gripper_joint_offset_y} ${right_gripper_joint_offset_z}" />
+    <origin rpy="0 0 0" xyz="${pad_joint_offset_x} ${pad_joint_offset_y} ${pad_joint_offset_z}"/>
+    <parent link="right_gripper_tube"/>
+    <child link="right_gripper_pad_with_base"/>
+    <axis xyz="0 1 0"/>
+    <limit lower="-1.58" upper="1.58" effort="0" velocity="0.68"/>
+  </joint>
+  <joint name="right_gripper_finger_yaw_joint" type="revolute">
+    <origin rpy="0 0 0" xyz="${finger_base_offset_x} ${l_finger_base_offset_y} ${finger_base_offset_z}"/>
     <parent link="right_gripper_base"/>
-    <child link="right_gripper_vacuum_pad_base"/>
-    <axis xyz="0 1 0"/>
-    <limit lower="-1.58" upper="1.58" effort="0" velocity="4.5"/>
+    <child link="right_gripper_l_finger_base"/>
+    <axis xyz="0 0 1"/>
+    <limit lower="0" upper="1.58" effort="0" velocity="0.66"/>
   </joint>
-  <joint name="right_gripper_vacuum_pad_fixed" type="fixed">
+  <joint name="right_gripper_r_finger_yaw_joint" type="revolute">
+    <origin rpy="0 0 0" xyz="${finger_base_offset_x} ${r_finger_base_offset_y} ${finger_base_offset_z}"/>
+    <parent link="right_gripper_base"/>
+    <child link="right_gripper_r_finger_base"/>
+    <mimic joint="right_gripper_finger_yaw_joint" multiplier="1"/>
+    <axis xyz="0 0 -1"/>
+    <limit lower="0" upper="1.58" effort="0" velocity="0.66"/>
+  </joint>
+  <joint name="right_gripper_finger_roll_joint" type="revolute">
     <origin rpy="0 0 0" xyz="0 0 0"/>
-    <parent link="right_gripper_vacuum_pad_base"/>
-    <child link="right_gripper_vacuum_pad"/>
+    <parent link="right_gripper_l_finger_base"/>
+    <child link="right_gripper_l_finger"/>
+    <axis xyz="1 0 0"/>
+    <limit lower="0" upper="3.14" effort="0" velocity="1.0"/>
+  </joint>
+  <joint name="right_gripper_r_finger_roll_joint" type="revolute">
+    <origin rpy="0 0 0" xyz="0 0 0"/>
+    <parent link="right_gripper_r_finger_base"/>
+    <child link="right_gripper_r_finger"/>
+    <mimic joint="right_gripper_finger_roll_joint" multiplier="1"/>
+    <axis xyz="-1 0 0"/>
+    <limit lower="0" upper="3.14" effort="0" velocity="1.0"/>
   </joint>
 </robot>

Commit message: Add transmission to right_vacuum_gripper.xacro

File: jsk_2016_01_baxter_apc/robots/right_vacuum_gripper.xacro (robot description, xacro)
@@ -151,3 +151,44 @@
     <limit lower="0" upper="3.14" effort="0" velocity="1.0"/>
   </joint>
+  <!--Transmission-->
+  <transmission name="right_gripper_prismatic_trans">
+    <type>transmission_interface/SimpleTransmission</type>
+    <joint name="right_gripper_prismatic_joint">
+      <hardwareInterface>PositionJointInterface</hardwareInterface>
+    </joint>
+    <actuator name="right_gripper_prismatic_joint_motor">
+      <hardwareInterface>PositionJointInterface</hardwareInterface>
+      <mechanicalReduction>0.024</mechanicalReduction>
+    </actuator>
+  </transmission>
+  <transmission name="right_gripper_vacuum_pad_trans">
+    <type>transmission_interface/SimpleTransmission</type>
+    <joint name="right_gripper_vacuum_pad_joint">
+      <hardwareInterface>PositionJointInterface</hardwareInterface>
+    </joint>
+    <actuator name="right_gripper_vacuum_pad_tendon_winder">
+      <hardwareInterface>PositionJointInterface</hardwareInterface>
+      <mechanicalReduction>1.46484375</mechanicalReduction>
+    </actuator>
+  </transmission>
+  <transmission name="right_gripper_finger_yaw_trans">
+    <type>transmission_interface/SimpleTransmission</type>
+    <joint name="right_gripper_finger_yaw_joint">
+      <hardwareInterface>PositionJointInterface</hardwareInterface>
+    </joint>
+    <actuator name="right_gripper_finger_yaw_joint_motor">
+      <hardwareInterface>PositionJointInterface</hardwareInterface>
+      <mechanicalReduction>1.5</mechanicalReduction>
+    </actuator>
+  </transmission>
+  <transmission name="right_gripper_finger_roll_trans">
+    <type>transmission_interface/SimpleTransmission</type>
+    <joint name="right_gripper_finger_roll_joint">
+      <hardwareInterface>PositionJointInterface</hardwareInterface>
+    </joint>
+    <actuator name="right_gripper_finger_tendon_winder">
+      <hardwareInterface>PositionJointInterface</hardwareInterface>
+      <mechanicalReduction>1.0</mechanicalReduction>
+    </actuator>
+  </transmission>
 </robot>

Commit message: Add transmission to right_vacuum_gripper.xacro

File: jsk_2016_01_baxter_apc/robots/right_vacuum_gripper.xacro (robot description, xacro)
@@ -164,3 +164,44 @@
     <limit lower="0" upper="3.14" effort="0" velocity="1.0"/>
   </joint>
+  <!--Transmission-->
+  <transmission name="right_gripper_prismatic_trans">
+    <type>transmission_interface/SimpleTransmission</type>
+    <joint name="right_gripper_prismatic_joint">
+      <hardwareInterface>PositionJointInterface</hardwareInterface>
+    </joint>
+    <actuator name="right_gripper_prismatic_joint_motor">
+      <hardwareInterface>PositionJointInterface</hardwareInterface>
+      <mechanicalReduction>0.024</mechanicalReduction>
+    </actuator>
+  </transmission>
+  <transmission name="right_gripper_vacuum_pad_trans">
+    <type>transmission_interface/SimpleTransmission</type>
+    <joint name="right_gripper_vacuum_pad_joint">
+      <hardwareInterface>PositionJointInterface</hardwareInterface>
+    </joint>
+    <actuator name="right_gripper_vacuum_pad_tendon_winder">
+      <hardwareInterface>PositionJointInterface</hardwareInterface>
+      <mechanicalReduction>1.46484375</mechanicalReduction>
+    </actuator>
+  </transmission>
+  <transmission name="right_gripper_finger_yaw_trans">
+    <type>transmission_interface/SimpleTransmission</type>
+    <joint name="right_gripper_finger_yaw_joint">
+      <hardwareInterface>PositionJointInterface</hardwareInterface>
+    </joint>
+    <actuator name="right_gripper_finger_yaw_joint_motor">
+      <hardwareInterface>PositionJointInterface</hardwareInterface>
+      <mechanicalReduction>1.5</mechanicalReduction>
+    </actuator>
+  </transmission>
+  <transmission name="right_gripper_finger_roll_trans">
+    <type>transmission_interface/SimpleTransmission</type>
+    <joint name="right_gripper_finger_roll_joint">
+      <hardwareInterface>PositionJointInterface</hardwareInterface>
+    </joint>
+    <actuator name="right_gripper_finger_tendon_winder">
+      <hardwareInterface>PositionJointInterface</hardwareInterface>
+      <mechanicalReduction>1.0</mechanicalReduction>
+    </actuator>
+  </transmission>
 </robot>

Commit message: Add right gripper-v5 collision

File: jsk_2016_01_baxter_apc/robots/right_vacuum_gripper.xacro (robot description, xacro)
@@ -16,7 +16,33 @@
   </gazebo>
   <!--Link bodies-->
+  <xacro:property name="base_rect_offset_x" value="0.0065" />
+  <xacro:property name="base_rect_l" value="0.2805" />
+  <xacro:property name="base_rect_h" value="0.107" />
+  <xacro:property name="base_rect_w" value="0.15" />
+  <xacro:property name="camera_rect_offset_x" value="-0.061" />
+  <xacro:property name="camera_rect_offset_y" value="-0.037" />
+  <xacro:property name="camera_rect_offset_z" value="0.004" />
+  <xacro:property name="camera_rect_l" value="0.04" />
+  <xacro:property name="camera_rect_h" value="0.03" />
+  <xacro:property name="camera_rect_w" value="0.165" />
+  <xacro:property name="tube_rect_offset_x" value="0.0475" />
+  <xacro:property name="tube_rect_offset_y" value="0.012" />
+  <xacro:property name="tube_rect_offset_z" value="0.17" />
+  <xacro:property name="tube_rect_l" value="0.29" />
+  <xacro:property name="tube_rect_h" value="0.034" />
+  <xacro:property name="tube_rect_w" value="0.081" />
   <xacro:property name="pad_with_base_offset_x" value="-0.048" />
   <xacro:property name="pad_with_base_offset_y" value="-0.0005" />
   <xacro:property name="pad_with_base_offset_z" value="-0.302" />
+  <xacro:property name="pad_with_base_col_z" value="0.0145" />
+  <xacro:property name="pad_with_base_rect_l" value="0.055" />
+  <xacro:property name="pad_with_base_rect_h" value="0.028" />
+  <xacro:property name="pad_with_base_rect_w" value="0.028" />
+  <xacro:property name="finger_base_rect_l" value="0.022" />
+  <xacro:property name="finger_base_rect_h" value="0.032" />
+  <xacro:property name="finger_base_rect_w" value="0.036" />
+  <xacro:property name="finger_rect_l" value="0.04" />
+  <xacro:property name="finger_rect_h" value="0.016" />
+  <xacro:property name="finger_rect_w" value="0.11" />
   <!--Joints-->
   <xacro:property name="hand_offset_x" value="-0.01" />
@@ -40,5 +66,16 @@
       </material>
     </visual>
-    <!--FIXME: Add collision-->
+    <collision>
+      <origin rpy="0 0 0" xyz="${base_rect_offset_x} 0 ${base_rect_l/2}"/>
+      <geometry>
+        <box size="${base_rect_h} ${base_rect_w} ${base_rect_l}"/>
+      </geometry>
+    </collision>
+    <collision>
+      <origin rpy="0 0 0" xyz="${camera_rect_offset_x} ${camera_rect_offset_y} ${camera_rect_offset_z}"/>
+      <geometry>
+        <box size="${camera_rect_h} ${camera_rect_w} ${camera_rect_l}"/>
+      </geometry>
+    </collision>
   </link>
   <link name="right_gripper_tube">
@@ -52,5 +89,10 @@
       </material>
     </visual>
-    <!--FIXME: Add collision-->
+    <collision>
+      <origin rpy="0 0 0" xyz="${tube_rect_offset_x} ${tube_rect_offset_y} ${tube_rect_offset_z}"/>
+      <geometry>
+        <box size="${tube_rect_h} ${tube_rect_w} ${tube_rect_l}"/>
+      </geometry>
+    </collision>
   </link>
   <link name="right_gripper_pad_with_base">
@@ -64,5 +106,10 @@
       </material>
     </visual>
-    <!--FIXME: Add collision-->
+    <collision>
+      <origin rpy="0 0 0" xyz="0 0 ${pad_with_base_col_z}"/>
+      <geometry>
+        <box size="${pad_with_base_rect_h} ${pad_with_base_rect_w} ${pad_with_base_rect_l}"/>
+      </geometry>
+    </collision>
   </link>
   <link name="right_gripper_r_finger_base">
@@ -76,5 +123,10 @@
       </material>
     </visual>
-    <!--FIXME: Add collision-->
+    <collision>
+      <origin rpy="0 0 0" xyz="0 0 ${-finger_base_rect_l/2}"/>
+      <geometry>
+        <box size="${finger_base_rect_h} ${finger_base_rect_w} ${finger_base_rect_l}"/>
+      </geometry>
+    </collision>
   </link>
   <link name="right_gripper_l_finger_base">
@@ -88,5 +140,10 @@
       </material>
     </visual>
-    <!--FIXME: Add collision-->
+    <collision>
+      <origin rpy="0 0 0" xyz="0 0 ${-finger_base_rect_l/2}"/>
+      <geometry>
+        <box size="${finger_base_rect_h} ${finger_base_rect_w} ${finger_base_rect_l}"/>
+      </geometry>
+    </collision>
   </link>
   <link name="right_gripper_r_finger">
@@ -100,5 +157,10 @@
       </material>
     </visual>
-    <!--FIXME: Add collision-->
+    <collision>
+      <origin rpy="0 0 0" xyz="0 ${-finger_rect_w/2} 0"/>
+      <geometry>
+        <box size="${finger_rect_h} ${finger_rect_w} ${finger_rect_l}"/>
+      </geometry>
+    </collision>
   </link>
   <link name="right_gripper_l_finger">
@@ -112,5 +174,10 @@
       </material>
     </visual>
-    <!--FIXME: Add collision-->
+    <collision>
+      <origin rpy="0 0 0" xyz="0 ${finger_rect_w/2} 0"/>
+      <geometry>
+        <box size="${finger_rect_h} ${finger_rect_w} ${finger_rect_l}"/>
+      </geometry>
+    </collision>
   </link>
   <!--Joints-->
