Commit message: Add right gripper-v5 collision

File: jsk_2016_01_baxter_apc/robots/right_vacuum_gripper.xacro (robot description, xacro)
@@ -3,7 +3,33 @@
   <xacro:include filename="$(find jsk_2016_01_baxter_apc)/robots/common_constants.xacro"/>
   <!--Link bodies-->
+  <xacro:property name="base_rect_offset_x" value="0.0065" />
+  <xacro:property name="base_rect_l" value="0.2805" />
+  <xacro:property name="base_rect_h" value="0.107" />
+  <xacro:property name="base_rect_w" value="0.15" />
+  <xacro:property name="camera_rect_offset_x" value="-0.061" />
+  <xacro:property name="camera_rect_offset_y" value="-0.037" />
+  <xacro:property name="camera_rect_offset_z" value="0.004" />
+  <xacro:property name="camera_rect_l" value="0.04" />
+  <xacro:property name="camera_rect_h" value="0.03" />
+  <xacro:property name="camera_rect_w" value="0.165" />
+  <xacro:property name="tube_rect_offset_x" value="0.0475" />
+  <xacro:property name="tube_rect_offset_y" value="0.012" />
+  <xacro:property name="tube_rect_offset_z" value="0.17" />
+  <xacro:property name="tube_rect_l" value="0.29" />
+  <xacro:property name="tube_rect_h" value="0.034" />
+  <xacro:property name="tube_rect_w" value="0.081" />
   <xacro:property name="pad_with_base_offset_x" value="-0.048" />
   <xacro:property name="pad_with_base_offset_y" value="-0.0005" />
   <xacro:property name="pad_with_base_offset_z" value="-0.302" />
+  <xacro:property name="pad_with_base_col_z" value="0.0145" />
+  <xacro:property name="pad_with_base_rect_l" value="0.055" />
+  <xacro:property name="pad_with_base_rect_h" value="0.028" />
+  <xacro:property name="pad_with_base_rect_w" value="0.028" />
+  <xacro:property name="finger_base_rect_l" value="0.022" />
+  <xacro:property name="finger_base_rect_h" value="0.032" />
+  <xacro:property name="finger_base_rect_w" value="0.036" />
+  <xacro:property name="finger_rect_l" value="0.04" />
+  <xacro:property name="finger_rect_h" value="0.016" />
+  <xacro:property name="finger_rect_w" value="0.11" />
   <!--Joints-->
   <xacro:property name="hand_offset_x" value="-0.01" />
@@ -27,5 +53,16 @@
       </material>
     </visual>
-    <!--FIXME: Add collision-->
+    <collision>
+      <origin rpy="0 0 0" xyz="${base_rect_offset_x} 0 ${base_rect_l/2}"/>
+      <geometry>
+        <box size="${base_rect_h} ${base_rect_w} ${base_rect_l}"/>
+      </geometry>
+    </collision>
+    <collision>
+      <origin rpy="0 0 0" xyz="${camera_rect_offset_x} ${camera_rect_offset_y} ${camera_rect_offset_z}"/>
+      <geometry>
+        <box size="${camera_rect_h} ${camera_rect_w} ${camera_rect_l}"/>
+      </geometry>
+    </collision>
   </link>
   <link name="right_gripper_tube">
@@ -39,5 +76,10 @@
       </material>
     </visual>
-    <!--FIXME: Add collision-->
+    <collision>
+      <origin rpy="0 0 0" xyz="${tube_rect_offset_x} ${tube_rect_offset_y} ${tube_rect_offset_z}"/>
+      <geometry>
+        <box size="${tube_rect_h} ${tube_rect_w} ${tube_rect_l}"/>
+      </geometry>
+    </collision>
   </link>
   <link name="right_gripper_pad_with_base">
@@ -51,5 +93,10 @@
       </material>
     </visual>
-    <!--FIXME: Add collision-->
+    <collision>
+      <origin rpy="0 0 0" xyz="0 0 ${pad_with_base_col_z}"/>
+      <geometry>
+        <box size="${pad_with_base_rect_h} ${pad_with_base_rect_w} ${pad_with_base_rect_l}"/>
+      </geometry>
+    </collision>
   </link>
   <link name="right_gripper_r_finger_base">
@@ -63,5 +110,10 @@
       </material>
     </visual>
-    <!--FIXME: Add collision-->
+    <collision>
+      <origin rpy="0 0 0" xyz="0 0 ${-finger_base_rect_l/2}"/>
+      <geometry>
+        <box size="${finger_base_rect_h} ${finger_base_rect_w} ${finger_base_rect_l}"/>
+      </geometry>
+    </collision>
   </link>
   <link name="right_gripper_l_finger_base">
@@ -75,5 +127,10 @@
       </material>
     </visual>
-    <!--FIXME: Add collision-->
+    <collision>
+      <origin rpy="0 0 0" xyz="0 0 ${-finger_base_rect_l/2}"/>
+      <geometry>
+        <box size="${finger_base_rect_h} ${finger_base_rect_w} ${finger_base_rect_l}"/>
+      </geometry>
+    </collision>
   </link>
   <link name="right_gripper_r_finger">
@@ -87,5 +144,10 @@
       </material>
     </visual>
-    <!--FIXME: Add collision-->
+    <collision>
+      <origin rpy="0 0 0" xyz="0 ${-finger_rect_w/2} 0"/>
+      <geometry>
+        <box size="${finger_rect_h} ${finger_rect_w} ${finger_rect_l}"/>
+      </geometry>
+    </collision>
   </link>
   <link name="right_gripper_l_finger">
@@ -99,5 +161,10 @@
       </material>
     </visual>
-    <!--FIXME: Add collision-->
+    <collision>
+      <origin rpy="0 0 0" xyz="0 ${finger_rect_w/2} 0"/>
+      <geometry>
+        <box size="${finger_rect_h} ${finger_rect_w} ${finger_rect_l}"/>
+      </geometry>
+    </collision>
   </link>
   <!--Joints-->

Commit message: Add calib_speed and increase joint speed

File: jsk_2016_01_baxter_apc/robots/right_vacuum_gripper.xacro (robot description, xacro)
@@ -192,5 +192,5 @@
     <child link="right_gripper_tube"/>
     <axis xyz="0 0 1"/>
-    <limit lower="0" upper="0.124" effort="0" velocity="0.024"/>
+    <limit lower="0" upper="0.124" effort="0" velocity="0.048"/>
   </joint>
   <joint name="right_gripper_vacuum_pad_joint" type="revolute">

Commit message: Add calib_speed and increase joint speed

File: jsk_2016_01_baxter_apc/robots/right_vacuum_gripper.xacro (robot description, xacro)
@@ -179,5 +179,5 @@
     <child link="right_gripper_tube"/>
     <axis xyz="0 0 1"/>
-    <limit lower="0" upper="0.124" effort="0" velocity="0.024"/>
+    <limit lower="0" upper="0.124" effort="0" velocity="0.048"/>
   </joint>
   <joint name="right_gripper_vacuum_pad_joint" type="revolute">

Commit message: Maximize gripper joint speed

File: jsk_2016_01_baxter_apc/robots/right_vacuum_gripper.xacro (robot description, xacro)
@@ -199,5 +199,5 @@
     <child link="right_gripper_pad_with_base"/>
     <axis xyz="0 1 0"/>
-    <limit lower="-1.58" upper="1.58" effort="0" velocity="0.68"/>
+    <limit lower="-1.58" upper="1.58" effort="0" velocity="2.24"/>
   </joint>
   <joint name="right_gripper_finger_yaw_joint" type="revolute">
@@ -206,5 +206,5 @@
     <child link="right_gripper_l_finger_base"/>
     <axis xyz="0 0 1"/>
-    <limit lower="0" upper="1.58" effort="0" velocity="0.66"/>
+    <limit lower="0" upper="1.58" effort="0" velocity="0.76"/>
   </joint>
   <joint name="right_gripper_r_finger_yaw_joint" type="revolute">
@@ -214,5 +214,5 @@
     <mimic joint="right_gripper_finger_yaw_joint" multiplier="1"/>
     <axis xyz="0 0 -1"/>
-    <limit lower="0" upper="1.58" effort="0" velocity="0.66"/>
+    <limit lower="0" upper="1.58" effort="0" velocity="0.76"/>
   </joint>
   <joint name="right_gripper_finger_roll_joint" type="revolute">
@@ -221,5 +221,5 @@
     <child link="right_gripper_l_finger"/>
     <axis xyz="1 0 0"/>
-    <limit lower="0" upper="3.14" effort="0" velocity="1.0"/>
+    <limit lower="0" upper="3.14" effort="0" velocity="3.0"/>
   </joint>
   <joint name="right_gripper_r_finger_roll_joint" type="revolute">
@@ -229,5 +229,5 @@
     <mimic joint="right_gripper_finger_roll_joint" multiplier="1"/>
     <axis xyz="-1 0 0"/>
-    <limit lower="0" upper="3.14" effort="0" velocity="1.0"/>
+    <limit lower="0" upper="3.14" effort="0" velocity="3.0"/>
   </joint>
   <!--Transmission-->
