Commit message: use smaller collision head

File: jsk_2016_01_baxter_apc/robots/baxter_simple.urdf (robot description, URDF)
Before this commit: robot baxter, 45 links, 44 joints
Links:
- link collision_head_link_1: geometry collision sphere radius=0.1; visual sphere radius=0.001
- link collision_head_link_2: geometry collision sphere radius=0.1; visual sphere radius=0.001
