Commit message: tf publish frame of cameras separately from xacro

File: jsk_2016_01_baxter_apc/robots/softkinetic_camera/senz3d.urdf.xacro (robot description, xacro)
@@ -43,7 +43,7 @@
       <origin xyz="0.0 0.0 0.0" rpy="${-M_PI/2} 0.0 ${-M_PI/2}"/>
       <parent link="${name}_rgb_frame"/>
-      <child link="${name}_rgb_optical_frame"/>
+      <child link="${name}_rgb_optical_frame_base"/>
     </joint>
-    <link name="${name}_rgb_optical_frame"/>
+    <link name="${name}_rgb_optical_frame_base"/>
     <joint name="${name}_depth_joint" type="fixed">
       <origin xyz="0.0 -0.0125 0.0" rpy="0.0 0.0 0.0"/>
