Commit message: update right_vacuum_gripper.xacro for gazebo

File: jsk_arc2017_baxter/robots/right_vacuum_gripper.xacro (robot description, xacro)
@@ -5,15 +5,34 @@
   <gazebo reference="right_gripper_base">
     <selfCollide>true</selfCollide>
-    <material>Gazebo/White</material>
-  </gazebo>
-  <gazebo reference="right_gripper_vacuum_pad_base">
+    <material>Gazebo/Black</material>
+  </gazebo>
+  <gazebo reference="right_gripper_tube">
     <selfCollide>true</selfCollide>
     <material>Gazebo/Grey</material>
   </gazebo>
-  <gazebo reference="right_gripper_vacuum_pad">
+  <gazebo reference="right_gripper_pad_with_base">
     <selfCollide>true</selfCollide>
     <material>Gazebo/Green</material>
   </gazebo>
+  <gazebo reference="right_gripper_l_finger_base">
+    <selfCollide>true</selfCollide>
+    <material>Gazebo/Black</material>
+  </gazebo>
+  <gazebo reference="right_gripper_r_finger_base">
+    <selfCollide>true</selfCollide>
+    <material>Gazebo/Black</material>
+  </gazebo>
+  <gazebo reference="right_gripper_l_finger">
+    <selfCollide>true</selfCollide>
+    <material>Gazebo/Black</material>
+  </gazebo>
+  <gazebo reference="right_gripper_r_finger">
+    <selfCollide>true</selfCollide>
+    <material>Gazebo/Black</material>
+  </gazebo>
   <gazebo reference="right_gripper_vacuum_pad_joint">
+    <implicitSpringDamper>false</implicitSpringDamper>
+  </gazebo>
+  <gazebo reference="right_gripper_prismatic_joint">
     <implicitSpringDamper>false</implicitSpringDamper>
   </gazebo>
@@ -295,4 +314,5 @@
     <axis xyz="0 0 1"/>
     <limit lower="0" upper="0.124" effort="0" velocity="0.132"/>
+    <dynamics damping="0.7"/>
   </joint>
   <joint name="right_gripper_vacuum_pad_joint" type="revolute">
