Commit message: add damping to gripper joints

File: jsk_arc2017_baxter/robots/left_vacuum_gripper.xacro (robot description, xacro)
@@ -307,4 +307,5 @@
     <parent link="left_hand"/>
     <child link="left_gripper_base"/>
+    <dynamics damping="0.7"/>
   </joint>
   <joint name="left_gripper_prismatic_joint" type="prismatic">
@@ -322,4 +323,5 @@
     <axis xyz="0 1 0"/>
     <limit lower="-1.58" upper="1.58" effort="0" velocity="3.36"/>
+    <dynamics damping="0.7"/>
   </joint>
   <joint name="left_gripper_finger_yaw_joint" type="revolute">
@@ -329,4 +331,5 @@
     <axis xyz="0 0 1"/>
     <limit lower="0" upper="1.58" effort="0" velocity="4.23"/>
+    <dynamics damping="0.7"/>
   </joint>
   <joint name="left_gripper_r_finger_yaw_joint" type="revolute">
@@ -337,4 +340,5 @@
     <axis xyz="0 0 -1"/>
     <limit lower="0" upper="1.58" effort="0" velocity="4.23"/>
+    <dynamics damping="0.7"/>
   </joint>
   <joint name="left_gripper_finger_roll_joint" type="revolute">
@@ -344,4 +348,5 @@
     <axis xyz="1 0 0"/>
     <limit lower="0" upper="3.14" effort="0" velocity="5.5"/>
+    <dynamics damping="0.7"/>
   </joint>
   <joint name="left_gripper_r_finger_roll_joint" type="revolute">
@@ -352,4 +357,5 @@
     <axis xyz="-1 0 0"/>
     <limit lower="0" upper="3.14" effort="0" velocity="5.5"/>
+    <dynamics damping="0.7"/>
   </joint>
   <joint name="left_gripper_palm_endpoint_fixed" type="fixed">

File: jsk_arc2017_baxter/robots/right_vacuum_gripper.xacro (robot description, xacro)
@@ -322,4 +322,5 @@
     <axis xyz="0 1 0"/>
     <limit lower="-1.58" upper="1.58" effort="0" velocity="3.36"/>
+    <dynamics damping="0.7"/>
   </joint>
   <joint name="right_gripper_finger_yaw_joint" type="revolute">
@@ -329,4 +330,5 @@
     <axis xyz="0 0 1"/>
     <limit lower="0" upper="1.58" effort="0" velocity="4.23"/>
+    <dynamics damping="0.7"/>
   </joint>
   <joint name="right_gripper_r_finger_yaw_joint" type="revolute">
@@ -337,4 +339,5 @@
     <axis xyz="0 0 -1"/>
     <limit lower="0" upper="1.58" effort="0" velocity="4.23"/>
+    <dynamics damping="0.7"/>
   </joint>
   <joint name="right_gripper_finger_roll_joint" type="revolute">
@@ -344,4 +347,5 @@
     <axis xyz="1 0 0"/>
     <limit lower="0" upper="3.14" effort="0" velocity="5.5"/>
+    <dynamics damping="0.7"/>
   </joint>
   <joint name="right_gripper_r_finger_roll_joint" type="revolute">
@@ -352,4 +356,5 @@
     <axis xyz="-1 0 0"/>
     <limit lower="0" upper="3.14" effort="0" velocity="5.5"/>
+    <dynamics damping="0.7"/>
   </joint>
   <joint name="right_gripper_palm_endpoint_fixed" type="fixed">

Commit message: Avoid name clashes of properties in baxter

File: jsk_arc2017_baxter/robots/left_vacuum_gripper.xacro (robot description, xacro)
@@ -38,45 +38,45 @@
   </gazebo>
   <!--Link bodies-->
-  <xacro:property name="base_rect_offset_x" value="0.0065" />
-  <xacro:property name="base_rect_l" value="0.2805" />
-  <xacro:property name="base_rect_h" value="0.107" />
-  <xacro:property name="base_rect_w" value="0.15" />
-  <xacro:property name="camera_rect_offset_x" value="-0.061" />
-  <xacro:property name="camera_rect_offset_y" value="0.037" />
-  <xacro:property name="camera_rect_offset_z" value="0.004" />
-  <xacro:property name="camera_rect_l" value="0.04" />
-  <xacro:property name="camera_rect_h" value="0.03" />
-  <xacro:property name="camera_rect_w" value="0.165" />
-  <xacro:property name="tube_rect_offset_x" value="0.0475" />
-  <xacro:property name="tube_rect_offset_y" value="-0.012" />
-  <xacro:property name="tube_rect_offset_z" value="0.17" />
-  <xacro:property name="tube_rect_l" value="0.29" />
-  <xacro:property name="tube_rect_h" value="0.034" />
-  <xacro:property name="tube_rect_w" value="0.081" />
-  <xacro:property name="pad_with_base_offset_x" value="-0.048" />
-  <xacro:property name="pad_with_base_offset_y" value="0.0005" />
-  <xacro:property name="pad_with_base_offset_z" value="-0.302" />
-  <xacro:property name="pad_with_base_col_z" value="0.0145" />
-  <xacro:property name="pad_with_base_rect_l" value="0.055" />
-  <xacro:property name="pad_with_base_rect_h" value="0.028" />
-  <xacro:property name="pad_with_base_rect_w" value="0.028" />
-  <xacro:property name="finger_base_rect_l" value="0.022" />
-  <xacro:property name="finger_base_rect_h" value="0.032" />
-  <xacro:property name="finger_base_rect_w" value="0.036" />
-  <xacro:property name="finger_rect_l" value="0.04" />
-  <xacro:property name="finger_rect_h" value="0.016" />
-  <xacro:property name="finger_rect_w" value="0.11" />
+  <xacro:property name="lg_base_rect_offset_x" value="0.0065" />
+  <xacro:property name="lg_base_rect_l" value="0.2805" />
+  <xacro:property name="lg_base_rect_h" value="0.107" />
+  <xacro:property name="lg_base_rect_w" value="0.15" />
+  <xacro:property name="lg_camera_rect_offset_x" value="-0.061" />
+  <xacro:property name="lg_camera_rect_offset_y" value="0.037" />
+  <xacro:property name="lg_camera_rect_offset_z" value="0.004" />
+  <xacro:property name="lg_camera_rect_l" value="0.04" />
+  <xacro:property name="lg_camera_rect_h" value="0.03" />
+  <xacro:property name="lg_camera_rect_w" value="0.165" />
+  <xacro:property name="lg_tube_rect_offset_x" value="0.0475" />
+  <xacro:property name="lg_tube_rect_offset_y" value="-0.012" />
+  <xacro:property name="lg_tube_rect_offset_z" value="0.17" />
+  <xacro:property name="lg_tube_rect_l" value="0.29" />
+  <xacro:property name="lg_tube_rect_h" value="0.034" />
+  <xacro:property name="lg_tube_rect_w" value="0.081" />
+  <xacro:property name="lg_pad_with_base_offset_x" value="-0.048" />
+  <xacro:property name="lg_pad_with_base_offset_y" value="0.0005" />
+  <xacro:property name="lg_pad_with_base_offset_z" value="-0.302" />
+  <xacro:property name="lg_pad_with_base_col_z" value="0.0145" />
+  <xacro:property name="lg_pad_with_base_rect_l" value="0.055" />
+  <xacro:property name="lg_pad_with_base_rect_h" value="0.028" />
+  <xacro:property name="lg_pad_with_base_rect_w" value="0.028" />
+  <xacro:property name="lg_finger_base_rect_l" value="0.022" />
+  <xacro:property name="lg_finger_base_rect_h" value="0.032" />
+  <xacro:property name="lg_finger_base_rect_w" value="0.036" />
+  <xacro:property name="lg_finger_rect_l" value="0.04" />
+  <xacro:property name="lg_finger_rect_h" value="0.016" />
+  <xacro:property name="lg_finger_rect_w" value="0.11" />
   <!--Joints-->
-  <xacro:property name="hand_offset_x" value="-0.01" />
-  <xacro:property name="hand_offset_z" value="0" />
-  <xacro:property name="pad_joint_offset_x" value="0.048" />
-  <xacro:property name="pad_joint_offset_y" value="-0.0005" />
-  <xacro:property name="pad_joint_offset_z" value="0.302" />
-  <xacro:property name="finger_base_offset_z" value="0.291352" />
-  <xacro:property name="finger_base_offset_x" value="-0.014" />
-  <xacro:property name="l_finger_base_offset_y" value="0.026" />
-  <xacro:property name="r_finger_base_offset_y" value="-0.026" />
-  <xacro:property name="palm_offset_x" value="0.015" />
-  <xacro:property name="palm_offset_z" value="0.28" />
+  <xacro:property name="lg_hand_offset_x" value="-0.01" />
+  <xacro:property name="lg_hand_offset_z" value="0" />
+  <xacro:property name="lg_pad_joint_offset_x" value="0.048" />
+  <xacro:property name="lg_pad_joint_offset_y" value="-0.0005" />
+  <xacro:property name="lg_pad_joint_offset_z" value="0.302" />
+  <xacro:property name="lg_finger_base_offset_z" value="0.291352" />
+  <xacro:property name="lg_finger_base_offset_x" value="-0.014" />
+  <xacro:property name="lg_l_finger_base_offset_y" value="0.026" />
+  <xacro:property name="lg_r_finger_base_offset_y" value="-0.026" />
+  <xacro:property name="lg_palm_offset_x" value="0.015" />
+  <xacro:property name="lg_palm_offset_z" value="0.28" />
   <!--Link bodies-->
   <link name="left_gripper_base">
@@ -100,13 +100,13 @@
     </visual>
     <collision>
-      <origin rpy="0 0 0" xyz="${base_rect_offset_x} 0 ${base_rect_l/2}"/>
-      <geometry>
-        <box size="${base_rect_h} ${base_rect_w} ${base_rect_l}"/>
-      </geometry>
-    </collision>
-    <collision>
-      <origin rpy="0 0 0" xyz="${camera_rect_offset_x} ${camera_rect_offset_y} ${camera_rect_offset_z}"/>
-      <geometry>
-        <box size="${camera_rect_h} ${camera_rect_w} ${camera_rect_l}"/>
+      <origin rpy="0 0 0" xyz="${lg_base_rect_offset_x} 0 ${lg_base_rect_l/2}"/>
+      <geometry>
+        <box size="${lg_base_rect_h} ${lg_base_rect_w} ${lg_base_rect_l}"/>
+      </geometry>
+    </collision>
+    <collision>
+      <origin rpy="0 0 0" xyz="${lg_camera_rect_offset_x} ${lg_camera_rect_offset_y} ${lg_camera_rect_offset_z}"/>
+      <geometry>
+        <box size="${lg_camera_rect_h} ${lg_camera_rect_w} ${lg_camera_rect_l}"/>
       </geometry>
     </collision>
@@ -147,7 +147,7 @@
     </visual>
     <collision>
-      <origin rpy="0 0 0" xyz="${tube_rect_offset_x} ${tube_rect_offset_y} ${tube_rect_offset_z}"/>
-      <geometry>
-        <box size="${tube_rect_h} ${tube_rect_w} ${tube_rect_l}"/>
+      <origin rpy="0 0 0" xyz="${lg_tube_rect_offset_x} ${lg_tube_rect_offset_y} ${lg_tube_rect_offset_z}"/>
+      <geometry>
+        <box size="${lg_tube_rect_h} ${lg_tube_rect_w} ${lg_tube_rect_l}"/>
       </geometry>
     </collision>
@@ -161,5 +161,5 @@
   <link name="left_gripper_pad_with_base">
     <visual>
-      <origin rpy="${M_PI/2} 0 ${M_PI/2}" xyz="${pad_with_base_offset_x} ${pad_with_base_offset_y} ${pad_with_base_offset_z}"/>
+      <origin rpy="${M_PI/2} 0 ${M_PI/2}" xyz="${lg_pad_with_base_offset_x} ${lg_pad_with_base_offset_y} ${lg_pad_with_base_offset_z}"/>
       <geometry>
         <mesh filename="package://jsk_arc2017_baxter/meshes/gripper_v6/visual/left_gripper_vacuum_pad_base.stl" scale="0.001 0.001 0.001"/>
@@ -170,5 +170,5 @@
     </visual>
     <visual>
-      <origin rpy="${M_PI/2} 0 ${M_PI/2}" xyz="${pad_with_base_offset_x} ${pad_with_base_offset_y} ${pad_with_base_offset_z}"/>
+      <origin rpy="${M_PI/2} 0 ${M_PI/2}" xyz="${lg_pad_with_base_offset_x} ${lg_pad_with_base_offset_y} ${lg_pad_with_base_offset_z}"/>
       <geometry>
         <mesh filename="package://jsk_arc2017_baxter/meshes/gripper_v6/visual/left_gripper_vacuum_pad.stl" scale="0.001 0.001 0.001"/>
@@ -179,7 +179,7 @@
     </visual>
     <collision>
-      <origin rpy="0 0 0" xyz="0 0 ${pad_with_base_col_z}"/>
-      <geometry>
-        <box size="${pad_with_base_rect_h} ${pad_with_base_rect_w} ${pad_with_base_rect_l}"/>
+      <origin rpy="0 0 0" xyz="0 0 ${lg_pad_with_base_col_z}"/>
+      <geometry>
+        <box size="${lg_pad_with_base_rect_h} ${lg_pad_with_base_rect_w} ${lg_pad_with_base_rect_l}"/>
       </geometry>
     </collision>
@@ -202,7 +202,7 @@
     </visual>
     <collision>
-      <origin rpy="0 0 0" xyz="0 0 ${-finger_base_rect_l/2}"/>
-      <geometry>
-        <box size="${finger_base_rect_h} ${finger_base_rect_w} ${finger_base_rect_l}"/>
+      <origin rpy="0 0 0" xyz="0 0 ${-lg_finger_base_rect_l/2}"/>
+      <geometry>
+        <box size="${lg_finger_base_rect_h} ${lg_finger_base_rect_w} ${lg_finger_base_rect_l}"/>
       </geometry>
     </collision>
@@ -225,7 +225,7 @@
     </visual>
     <collision>
-      <origin rpy="0 0 0" xyz="0 0 ${-finger_base_rect_l/2}"/>
-      <geometry>
-        <box size="${finger_base_rect_h} ${finger_base_rect_w} ${finger_base_rect_l}"/>
+      <origin rpy="0 0 0" xyz="0 0 ${-lg_finger_base_rect_l/2}"/>
+      <geometry>
+        <box size="${lg_finger_base_rect_h} ${lg_finger_base_rect_w} ${lg_finger_base_rect_l}"/>
       </geometry>
     </collision>
@@ -257,7 +257,7 @@
     </visual>
     <collision>
-      <origin rpy="0 0 0" xyz="0 ${-finger_rect_w/2} 0"/>
-      <geometry>
-        <box size="${finger_rect_h} ${finger_rect_w} ${finger_rect_l}"/>
+      <origin rpy="0 0 0" xyz="0 ${-lg_finger_rect_w/2} 0"/>
+      <geometry>
+        <box size="${lg_finger_rect_h} ${lg_finger_rect_w} ${lg_finger_rect_l}"/>
       </geometry>
     </collision>
@@ -289,7 +289,7 @@
     </visual>
     <collision>
-      <origin rpy="0 0 0" xyz="0 ${finger_rect_w/2} 0"/>
-      <geometry>
-        <box size="${finger_rect_h} ${finger_rect_w} ${finger_rect_l}"/>
+      <origin rpy="0 0 0" xyz="0 ${lg_finger_rect_w/2} 0"/>
+      <geometry>
+        <box size="${lg_finger_rect_h} ${lg_finger_rect_w} ${lg_finger_rect_l}"/>
       </geometry>
     </collision>
@@ -304,5 +304,5 @@
   <!--Joints-->
   <joint name="left_gripper_base_fixed" type="fixed">
-    <origin rpy="0 0 0" xyz="${hand_offset_x} 0 ${hand_offset_z}" />
+    <origin rpy="0 0 0" xyz="${lg_hand_offset_x} 0 ${lg_hand_offset_z}" />
     <parent link="left_hand"/>
     <child link="left_gripper_base"/>
@@ -318,5 +318,5 @@
   </joint>
   <joint name="left_gripper_vacuum_pad_joint" type="revolute">
-    <origin rpy="0 0 0" xyz="${pad_joint_offset_x} ${pad_joint_offset_y} ${pad_joint_offset_z}"/>
+    <origin rpy="0 0 0" xyz="${lg_pad_joint_offset_x} ${lg_pad_joint_offset_y} ${lg_pad_joint_offset_z}"/>
     <parent link="left_gripper_tube"/>
     <child link="left_gripper_pad_with_base"/>
@@ -326,5 +326,5 @@
   </joint>
   <joint name="left_gripper_finger_yaw_joint" type="revolute">
-    <origin rpy="0 0 0" xyz="${finger_base_offset_x} ${l_finger_base_offset_y} ${finger_base_offset_z}"/>
+    <origin rpy="0 0 0" xyz="${lg_finger_base_offset_x} ${lg_l_finger_base_offset_y} ${lg_finger_base_offset_z}"/>
     <parent link="left_gripper_base"/>
     <child link="left_gripper_l_finger_base"/>
@@ -334,5 +334,5 @@
   </joint>
   <joint name="left_gripper_r_finger_yaw_joint" type="revolute">
-    <origin rpy="0 0 0" xyz="${finger_base_offset_x} ${r_finger_base_offset_y} ${finger_base_offset_z}"/>
+    <origin rpy="0 0 0" xyz="${lg_finger_base_offset_x} ${lg_r_finger_base_offset_y} ${lg_finger_base_offset_z}"/>
     <parent link="left_gripper_base"/>
     <child link="left_gripper_r_finger_base"/>
@@ -360,5 +360,5 @@
   </joint>
   <joint name="left_gripper_palm_endpoint_fixed" type="fixed">
-    <origin rpy="0 ${M_PI} 0" xyz="${palm_offset_x} 0 ${palm_offset_z}" />
+    <origin rpy="0 ${M_PI} 0" xyz="${lg_palm_offset_x} 0 ${lg_palm_offset_z}" />
     <parent link="left_gripper_base"/>
     <child link="left_gripper_palm_endpoint"/>
