Commit message: Avoid name clashes of properties in baxter

File: jsk_arc2017_baxter/robots/right_vacuum_gripper.xacro (robot description, xacro)
@@ -38,45 +38,45 @@
   </gazebo>
   <!--Link bodies-->
-  <xacro:property name="base_rect_offset_x" value="0.0065" />
-  <xacro:property name="base_rect_l" value="0.2805" />
-  <xacro:property name="base_rect_h" value="0.107" />
-  <xacro:property name="base_rect_w" value="0.15" />
-  <xacro:property name="camera_rect_offset_x" value="-0.061" />
-  <xacro:property name="camera_rect_offset_y" value="-0.037" />
-  <xacro:property name="camera_rect_offset_z" value="0.004" />
-  <xacro:property name="camera_rect_l" value="0.04" />
-  <xacro:property name="camera_rect_h" value="0.03" />
-  <xacro:property name="camera_rect_w" value="0.165" />
-  <xacro:property name="tube_rect_offset_x" value="0.0475" />
-  <xacro:property name="tube_rect_offset_y" value="0.012" />
-  <xacro:property name="tube_rect_offset_z" value="0.17" />
-  <xacro:property name="tube_rect_l" value="0.29" />
-  <xacro:property name="tube_rect_h" value="0.034" />
-  <xacro:property name="tube_rect_w" value="0.081" />
-  <xacro:property name="pad_with_base_offset_x" value="-0.048" />
-  <xacro:property name="pad_with_base_offset_y" value="-0.0005" />
-  <xacro:property name="pad_with_base_offset_z" value="-0.302" />
-  <xacro:property name="pad_with_base_col_z" value="0.0145" />
-  <xacro:property name="pad_with_base_rect_l" value="0.055" />
-  <xacro:property name="pad_with_base_rect_h" value="0.028" />
-  <xacro:property name="pad_with_base_rect_w" value="0.028" />
-  <xacro:property name="finger_base_rect_l" value="0.022" />
-  <xacro:property name="finger_base_rect_h" value="0.032" />
-  <xacro:property name="finger_base_rect_w" value="0.036" />
-  <xacro:property name="finger_rect_l" value="0.04" />
-  <xacro:property name="finger_rect_h" value="0.016" />
-  <xacro:property name="finger_rect_w" value="0.11" />
+  <xacro:property name="rg_base_rect_offset_x" value="0.0065" />
+  <xacro:property name="rg_base_rect_l" value="0.2805" />
+  <xacro:property name="rg_base_rect_h" value="0.107" />
+  <xacro:property name="rg_base_rect_w" value="0.15" />
+  <xacro:property name="rg_camera_rect_offset_x" value="-0.061" />
+  <xacro:property name="rg_camera_rect_offset_y" value="-0.037" />
+  <xacro:property name="rg_camera_rect_offset_z" value="0.004" />
+  <xacro:property name="rg_camera_rect_l" value="0.04" />
+  <xacro:property name="rg_camera_rect_h" value="0.03" />
+  <xacro:property name="rg_camera_rect_w" value="0.165" />
+  <xacro:property name="rg_tube_rect_offset_x" value="0.0475" />
+  <xacro:property name="rg_tube_rect_offset_y" value="0.012" />
+  <xacro:property name="rg_tube_rect_offset_z" value="0.17" />
+  <xacro:property name="rg_tube_rect_l" value="0.29" />
+  <xacro:property name="rg_tube_rect_h" value="0.034" />
+  <xacro:property name="rg_tube_rect_w" value="0.081" />
+  <xacro:property name="rg_pad_with_base_offset_x" value="-0.048" />
+  <xacro:property name="rg_pad_with_base_offset_y" value="-0.0005" />
+  <xacro:property name="rg_pad_with_base_offset_z" value="-0.302" />
+  <xacro:property name="rg_pad_with_base_col_z" value="0.0145" />
+  <xacro:property name="rg_pad_with_base_rect_l" value="0.055" />
+  <xacro:property name="rg_pad_with_base_rect_h" value="0.028" />
+  <xacro:property name="rg_pad_with_base_rect_w" value="0.028" />
+  <xacro:property name="rg_finger_base_rect_l" value="0.022" />
+  <xacro:property name="rg_finger_base_rect_h" value="0.032" />
+  <xacro:property name="rg_finger_base_rect_w" value="0.036" />
+  <xacro:property name="rg_finger_rect_l" value="0.04" />
+  <xacro:property name="rg_finger_rect_h" value="0.016" />
+  <xacro:property name="rg_finger_rect_w" value="0.11" />
   <!--Joints-->
-  <xacro:property name="hand_offset_x" value="-0.01" />
-  <xacro:property name="hand_offset_z" value="0" />
-  <xacro:property name="pad_joint_offset_x" value="0.048" />
-  <xacro:property name="pad_joint_offset_y" value="0.0005" />
-  <xacro:property name="pad_joint_offset_z" value="0.302" />
-  <xacro:property name="finger_base_offset_z" value="0.291352" />
-  <xacro:property name="finger_base_offset_x" value="-0.014" />
-  <xacro:property name="l_finger_base_offset_y" value="0.026" />
-  <xacro:property name="r_finger_base_offset_y" value="-0.026" />
-  <xacro:property name="palm_offset_x" value="0.015" />
-  <xacro:property name="palm_offset_z" value="0.28" />
+  <xacro:property name="rg_hand_offset_x" value="-0.01" />
+  <xacro:property name="rg_hand_offset_z" value="0" />
+  <xacro:property name="rg_pad_joint_offset_x" value="0.048" />
+  <xacro:property name="rg_pad_joint_offset_y" value="0.0005" />
+  <xacro:property name="rg_pad_joint_offset_z" value="0.302" />
+  <xacro:property name="rg_finger_base_offset_z" value="0.291352" />
+  <xacro:property name="rg_finger_base_offset_x" value="-0.014" />
+  <xacro:property name="rg_l_finger_base_offset_y" value="0.026" />
+  <xacro:property name="rg_r_finger_base_offset_y" value="-0.026" />
+  <xacro:property name="rg_palm_offset_x" value="0.015" />
+  <xacro:property name="rg_palm_offset_z" value="0.28" />
   <!--Link bodies-->
   <link name="right_gripper_base">
@@ -100,13 +100,13 @@
     </visual>
     <collision>
-      <origin rpy="0 0 0" xyz="${base_rect_offset_x} 0 ${base_rect_l/2}"/>
-      <geometry>
-        <box size="${base_rect_h} ${base_rect_w} ${base_rect_l}"/>
-      </geometry>
-    </collision>
-    <collision>
-      <origin rpy="0 0 0" xyz="${camera_rect_offset_x} ${camera_rect_offset_y} ${camera_rect_offset_z}"/>
-      <geometry>
-        <box size="${camera_rect_h} ${camera_rect_w} ${camera_rect_l}"/>
+      <origin rpy="0 0 0" xyz="${rg_base_rect_offset_x} 0 ${rg_base_rect_l/2}"/>
+      <geometry>
+        <box size="${rg_base_rect_h} ${rg_base_rect_w} ${rg_base_rect_l}"/>
+      </geometry>
+    </collision>
+    <collision>
+      <origin rpy="0 0 0" xyz="${rg_camera_rect_offset_x} ${rg_camera_rect_offset_y} ${rg_camera_rect_offset_z}"/>
+      <geometry>
+        <box size="${rg_camera_rect_h} ${rg_camera_rect_w} ${rg_camera_rect_l}"/>
       </geometry>
     </collision>
@@ -147,7 +147,7 @@
     </visual>
     <collision>
-      <origin rpy="0 0 0" xyz="${tube_rect_offset_x} ${tube_rect_offset_y} ${tube_rect_offset_z}"/>
-      <geometry>
-        <box size="${tube_rect_h} ${tube_rect_w} ${tube_rect_l}"/>
+      <origin rpy="0 0 0" xyz="${rg_tube_rect_offset_x} ${rg_tube_rect_offset_y} ${rg_tube_rect_offset_z}"/>
+      <geometry>
+        <box size="${rg_tube_rect_h} ${rg_tube_rect_w} ${rg_tube_rect_l}"/>
       </geometry>
     </collision>
@@ -161,5 +161,5 @@
   <link name="right_gripper_pad_with_base">
     <visual>
-      <origin rpy="${M_PI/2} 0 ${M_PI/2}" xyz="${pad_with_base_offset_x} ${pad_with_base_offset_y} ${pad_with_base_offset_z}"/>
+      <origin rpy="${M_PI/2} 0 ${M_PI/2}" xyz="${rg_pad_with_base_offset_x} ${rg_pad_with_base_offset_y} ${rg_pad_with_base_offset_z}"/>
       <geometry>
         <mesh filename="package://jsk_2016_01_baxter_apc/meshes/gripper-v5/visual/right_gripper_vacuum_pad_base.stl" scale="0.001 0.001 0.001"/>
@@ -170,5 +170,5 @@
     </visual>
     <visual>
-      <origin rpy="${M_PI/2} 0 ${M_PI/2}" xyz="${pad_with_base_offset_x} ${pad_with_base_offset_y} ${pad_with_base_offset_z}"/>
+      <origin rpy="${M_PI/2} 0 ${M_PI/2}" xyz="${rg_pad_with_base_offset_x} ${rg_pad_with_base_offset_y} ${rg_pad_with_base_offset_z}"/>
       <geometry>
         <mesh filename="package://jsk_2016_01_baxter_apc/meshes/gripper-v5/visual/right_gripper_vacuum_pad.stl" scale="0.001 0.001 0.001"/>
@@ -179,7 +179,7 @@
     </visual>
     <collision>
-      <origin rpy="0 0 0" xyz="0 0 ${pad_with_base_col_z}"/>
-      <geometry>
-        <box size="${pad_with_base_rect_h} ${pad_with_base_rect_w} ${pad_with_base_rect_l}"/>
+      <origin rpy="0 0 0" xyz="0 0 ${rg_pad_with_base_col_z}"/>
+      <geometry>
+        <box size="${rg_pad_with_base_rect_h} ${rg_pad_with_base_rect_w} ${rg_pad_with_base_rect_l}"/>
       </geometry>
     </collision>
@@ -202,7 +202,7 @@
     </visual>
     <collision>
-      <origin rpy="0 0 0" xyz="0 0 ${-finger_base_rect_l/2}"/>
-      <geometry>
-        <box size="${finger_base_rect_h} ${finger_base_rect_w} ${finger_base_rect_l}"/>
+      <origin rpy="0 0 0" xyz="0 0 ${-rg_finger_base_rect_l/2}"/>
+      <geometry>
+        <box size="${rg_finger_base_rect_h} ${rg_finger_base_rect_w} ${rg_finger_base_rect_l}"/>
       </geometry>
     </collision>
@@ -225,7 +225,7 @@
     </visual>
     <collision>
-      <origin rpy="0 0 0" xyz="0 0 ${-finger_base_rect_l/2}"/>
-      <geometry>
-        <box size="${finger_base_rect_h} ${finger_base_rect_w} ${finger_base_rect_l}"/>
+      <origin rpy="0 0 0" xyz="0 0 ${-rg_finger_base_rect_l/2}"/>
+      <geometry>
+        <box size="${rg_finger_base_rect_h} ${rg_finger_base_rect_w} ${rg_finger_base_rect_l}"/>
       </geometry>
     </collision>
@@ -257,7 +257,7 @@
     </visual>
     <collision>
-      <origin rpy="0 0 0" xyz="0 ${-finger_rect_w/2} 0"/>
-      <geometry>
-        <box size="${finger_rect_h} ${finger_rect_w} ${finger_rect_l}"/>
+      <origin rpy="0 0 0" xyz="0 ${-rg_finger_rect_w/2} 0"/>
+      <geometry>
+        <box size="${rg_finger_rect_h} ${rg_finger_rect_w} ${rg_finger_rect_l}"/>
       </geometry>
     </collision>
@@ -289,7 +289,7 @@
     </visual>
     <collision>
-      <origin rpy="0 0 0" xyz="0 ${finger_rect_w/2} 0"/>
-      <geometry>
-        <box size="${finger_rect_h} ${finger_rect_w} ${finger_rect_l}"/>
+      <origin rpy="0 0 0" xyz="0 ${rg_finger_rect_w/2} 0"/>
+      <geometry>
+        <box size="${rg_finger_rect_h} ${rg_finger_rect_w} ${rg_finger_rect_l}"/>
       </geometry>
     </collision>
@@ -304,5 +304,5 @@
   <!--Joints-->
   <joint name="right_gripper_base_fixed" type="fixed">
-    <origin rpy="0 0 0" xyz="${hand_offset_x} 0 ${hand_offset_z}" />
+    <origin rpy="0 0 0" xyz="${rg_hand_offset_x} 0 ${rg_hand_offset_z}" />
     <parent link="right_hand"/>
     <child link="right_gripper_base"/>
@@ -317,5 +317,5 @@
   </joint>
   <joint name="right_gripper_vacuum_pad_joint" type="revolute">
-    <origin rpy="0 0 0" xyz="${pad_joint_offset_x} ${pad_joint_offset_y} ${pad_joint_offset_z}"/>
+    <origin rpy="0 0 0" xyz="${rg_pad_joint_offset_x} ${rg_pad_joint_offset_y} ${rg_pad_joint_offset_z}"/>
     <parent link="right_gripper_tube"/>
     <child link="right_gripper_pad_with_base"/>
@@ -325,5 +325,5 @@
   </joint>
   <joint name="right_gripper_finger_yaw_joint" type="revolute">
-    <origin rpy="0 0 0" xyz="${finger_base_offset_x} ${l_finger_base_offset_y} ${finger_base_offset_z}"/>
+    <origin rpy="0 0 0" xyz="${rg_finger_base_offset_x} ${rg_l_finger_base_offset_y} ${rg_finger_base_offset_z}"/>
     <parent link="right_gripper_base"/>
     <child link="right_gripper_l_finger_base"/>
@@ -333,5 +333,5 @@
   </joint>
   <joint name="right_gripper_r_finger_yaw_joint" type="revolute">
-    <origin rpy="0 0 0" xyz="${finger_base_offset_x} ${r_finger_base_offset_y} ${finger_base_offset_z}"/>
+    <origin rpy="0 0 0" xyz="${rg_finger_base_offset_x} ${rg_r_finger_base_offset_y} ${rg_finger_base_offset_z}"/>
     <parent link="right_gripper_base"/>
     <child link="right_gripper_r_finger_base"/>
@@ -359,5 +359,5 @@
   </joint>
   <joint name="right_gripper_palm_endpoint_fixed" type="fixed">
-    <origin rpy="0 ${M_PI} 0" xyz="${palm_offset_x} 0 ${palm_offset_z}" />
+    <origin rpy="0 ${M_PI} 0" xyz="${rg_palm_offset_x} 0 ${rg_palm_offset_z}" />
     <parent link="right_gripper_base"/>
     <child link="right_gripper_palm_endpoint"/>
