Commit message: Use M_PI as joint limits in left gripper_v7

File: jsk_arc2017_baxter/robots/left_gripper_v7.xacro (robot description, xacro)
@@ -384,5 +384,5 @@
     <child link="left_gripper_pad_with_base"/>
     <axis xyz="0 1 0"/>
-    <limit lower="-1.58" upper="1.58" effort="0" velocity="3.36"/>
+    <limit lower="${-M_PI/2}" upper="${M_PI/2}" effort="0" velocity="3.36"/>
     <dynamics damping="0.7"/>
   </joint>
@@ -392,5 +392,5 @@
     <child link="left_gripper_r_finger_base"/>
     <axis xyz="0 0 1"/>
-    <limit lower="0" upper="1.58" effort="0" velocity="4.23"/>
+    <limit lower="0" upper="${M_PI/2}" effort="0" velocity="4.23"/>
     <dynamics damping="0.7"/>
   </joint>
@@ -401,5 +401,5 @@
     <mimic joint="left_gripper_finger_yaw_joint" multiplier="1"/>
     <axis xyz="0 0 -1"/>
-    <limit lower="0" upper="1.58" effort="0" velocity="4.23"/>
+    <limit lower="0" upper="${M_PI/2}" effort="0" velocity="4.23"/>
     <dynamics damping="0.7"/>
   </joint>
@@ -409,5 +409,5 @@
     <child link="left_gripper_l_finger_a"/>
     <axis xyz="1 0 0"/>
-    <limit lower="0" upper="1.57" effort="0" velocity="5.5"/>
+    <limit lower="0" upper="${M_PI/2}" effort="0" velocity="5.5"/>
     <dynamics damping="0.7"/>
   </joint>
@@ -418,5 +418,5 @@
     <mimic joint="left_gripper_finger_roll_joint_a" multiplier="1"/>
     <axis xyz="-1 0 0"/>
-    <limit lower="0" upper="1.57" effort="0" velocity="5.5"/>
+    <limit lower="0" upper="${M_PI/2}" effort="0" velocity="5.5"/>
     <dynamics damping="0.7"/>
   </joint>
@@ -426,5 +426,5 @@
     <child link="left_gripper_l_finger_bc"/>
     <axis xyz="1 0 0"/>
-    <limit lower="0" upper="3.14" effort="0" velocity="5.5"/>
+    <limit lower="0" upper="${M_PI}" effort="0" velocity="5.5"/>
     <dynamics damping="0.7"/>
   </joint>
@@ -435,5 +435,5 @@
     <mimic joint="left_gripper_finger_roll_joint_b" multiplier="1"/>
     <axis xyz="-1 0 0"/>
-    <limit lower="0" upper="3.14" effort="0" velocity="5.5"/>
+    <limit lower="0" upper="${M_PI}" effort="0" velocity="5.5"/>
     <dynamics damping="0.7"/>
   </joint>

Commit message: Fix collision of left gripper_v7

File: jsk_arc2017_baxter/robots/left_gripper_v7.xacro (robot description, xacro)
@@ -46,37 +46,37 @@
   </gazebo>
   <!--Link bodies-->
-  <xacro:property name="base_rect_offset_x" value="0.0065" />
-  <xacro:property name="base_rect_l" value="0.2805" />
-  <xacro:property name="base_rect_h" value="0.107" />
+  <xacro:property name="base_rect_offset_x" value="-0.023" />
+  <xacro:property name="base_rect_l" value="0.3036" />
+  <xacro:property name="base_rect_h" value="0.106" />
   <xacro:property name="base_rect_w" value="0.15" />
-  <xacro:property name="camera_rect_offset_x" value="-0.061" />
-  <xacro:property name="camera_rect_offset_y" value="0.037" />
+  <xacro:property name="camera_rect_offset_x" value="0.061" />
+  <xacro:property name="camera_rect_offset_y" value="-0.037" />
   <xacro:property name="camera_rect_offset_z" value="0.004" />
   <xacro:property name="camera_rect_l" value="0.04" />
   <xacro:property name="camera_rect_h" value="0.03" />
   <xacro:property name="camera_rect_w" value="0.165" />
-  <xacro:property name="tube_rect_offset_x" value="0.0475" />
-  <xacro:property name="tube_rect_offset_y" value="-0.012" />
-  <xacro:property name="tube_rect_offset_z" value="0.17" />
-  <xacro:property name="tube_rect_l" value="0.29" />
+  <xacro:property name="tube_rect_offset_x" value="-0.0515" />
+  <xacro:property name="tube_rect_offset_y" value="-0.00725" />
+  <xacro:property name="tube_rect_offset_z" value="0.1131" />
+  <xacro:property name="tube_rect_l" value="0.337" />
   <xacro:property name="tube_rect_h" value="0.034" />
-  <xacro:property name="tube_rect_w" value="0.081" />
+  <xacro:property name="tube_rect_w" value="0.0915" />
   <xacro:property name="pad_with_base_offset_x" value="0.0515" />
   <xacro:property name="pad_with_base_offset_y" value="0" />
   <xacro:property name="pad_with_base_offset_z" value="-0.2666" />
-  <xacro:property name="pad_with_base_col_z" value="0.0145" />
-  <xacro:property name="pad_with_base_rect_l" value="0.055" />
-  <xacro:property name="pad_with_base_rect_h" value="0.028" />
-  <xacro:property name="pad_with_base_rect_w" value="0.028" />
+  <xacro:property name="pad_with_base_col_z" value="0.0164" />
+  <xacro:property name="pad_with_base_rect_l" value="0.0628" />
+  <xacro:property name="pad_with_base_rect_h" value="0.0402" />
+  <xacro:property name="pad_with_base_rect_w" value="0.03" />
   <xacro:property name="finger_base_rect_l" value="0.022" />
   <xacro:property name="finger_base_rect_h" value="0.032" />
   <xacro:property name="finger_base_rect_w" value="0.036" />
-  <xacro:property name="finger_a_rect_l" value="0.028" />
+  <xacro:property name="finger_a_rect_l" value="0.036" />
   <xacro:property name="finger_a_rect_h" value="0.032" />
-  <xacro:property name="finger_a_rect_w" value="0.03" />
+  <xacro:property name="finger_a_rect_w" value="0.032" />
   <xacro:property name="l_finger_bc_offset_y" value="-0.022351" />
   <xacro:property name="r_finger_bc_offset_y" value="0.022351" />
   <xacro:property name="finger_bc_rect_l" value="0.11" />
-  <xacro:property name="finger_bc_rect_h" value="0.016" />
+  <xacro:property name="finger_bc_rect_h" value="0.0277" />
   <xacro:property name="finger_bc_rect_w" value="0.04" />
   <!--Joints-->
@@ -287,5 +287,5 @@
     </visual>
     <collision>
-      <origin rpy="0 0 0" xyz="0 ${finger_a_rect_w/2} 0"/>
+      <origin rpy="0 0 0" xyz="0 ${-finger_a_rect_w/2} 0"/>
       <geometry>
         <box size="${finger_a_rect_h} ${finger_a_rect_w} ${finger_a_rect_l}"/>
@@ -319,5 +319,5 @@
     </visual>
     <collision>
-      <origin rpy="0 0 0" xyz="0 ${finger_bc_rect_w/2} 0"/>
+      <origin rpy="0 0 0" xyz="0 0 ${-finger_bc_rect_l/2}"/>
       <geometry>
         <box size="${finger_bc_rect_h} ${finger_bc_rect_w} ${finger_bc_rect_l}"/>
@@ -351,5 +351,5 @@
     </visual>
     <collision>
-      <origin rpy="0 0 0" xyz="0 ${-finger_bc_rect_w/2} 0"/>
+      <origin rpy="0 0 0" xyz="0 0 ${-finger_bc_rect_l/2}"/>
       <geometry>
         <box size="${finger_bc_rect_h} ${finger_bc_rect_w} ${finger_bc_rect_l}"/>

Commit message: Use tendon transmission and fix hardwareInterface for real robot

File: jsk_arc2017_baxter/robots/left_gripper_v7.xacro (robot description, xacro)
@@ -444,11 +444,11 @@
   </joint>
   <!--Transmission-->
+  <!-- FIXME: In indigo, we may have to change hardwareInterface in gazebo -->
   <transmission name="left_gripper_prismatic_trans">
     <type>transmission_interface/SimpleTransmission</type>
     <joint name="left_gripper_prismatic_joint">
-      <hardwareInterface>PositionJointInterface</hardwareInterface>
+      <hardwareInterface>hardware_interface/PositionJointInterface</hardwareInterface>
     </joint>
     <actuator name="left_gripper_prismatic_joint_motor">
-      <hardwareInterface>PositionJointInterface</hardwareInterface>
       <mechanicalReduction>35.71428571</mechanicalReduction>  <!-- 1 / (0.8 * 35 * 0.001) -->
     </actuator>
@@ -457,8 +457,7 @@
     <type>transmission_interface/SimpleTransmission</type>
     <joint name="left_gripper_vacuum_pad_joint">
-      <hardwareInterface>PositionJointInterface</hardwareInterface>
+      <hardwareInterface>hardware_interface/PositionJointInterface</hardwareInterface>
     </joint>
     <actuator name="left_gripper_vacuum_pad_tendon_winder">
-      <hardwareInterface>PositionJointInterface</hardwareInterface>
       <mechanicalReduction>1.432291667</mechanicalReduction>
     </actuator>
@@ -467,20 +466,23 @@
     <type>transmission_interface/SimpleTransmission</type>
     <joint name="left_gripper_finger_yaw_joint">
-      <hardwareInterface>PositionJointInterface</hardwareInterface>
+      <hardwareInterface>hardware_interface/PositionJointInterface</hardwareInterface>
     </joint>
     <actuator name="left_gripper_finger_yaw_joint_motor">
-      <hardwareInterface>PositionJointInterface</hardwareInterface>
       <mechanicalReduction>1.5625</mechanicalReduction>  <!-- ~ 36 / 24 -->
     </actuator>
   </transmission>
-  <transmission name="left_gripper_finger_roll_trans">
-    <type>transmission_interface/SimpleTransmission</type>
+  <transmission name="left_gripper_finger_tendon_trans">
+    <type>jsk_arc2017_baxter/TendonTransmission</type>
+    <joint name="left_gripper_finger_roll_joint_a">
+      <hardwareInterface>hardware_interface/PositionJointInterface</hardwareInterface>
+      <limit>1.5707963268</limit>
+      <mechanicalReduction>1.0</mechanicalReduction>
+    </joint>
     <joint name="left_gripper_finger_roll_joint_b">
-      <hardwareInterface>PositionJointInterface</hardwareInterface>
+      <hardwareInterface>hardware_interface/PositionJointInterface</hardwareInterface>
+      <limit>3.14159265359</limit>
+      <mechanicalReduction>1.0</mechanicalReduction>
     </joint>
-    <actuator name="left_gripper_finger_tendon_winder">
-      <hardwareInterface>PositionJointInterface</hardwareInterface>
-      <mechanicalReduction>1.0</mechanicalReduction>
-    </actuator>
+    <actuator name="left_gripper_finger_tendon_winder" />
   </transmission>
 </robot>
