Commit message: Adjust moveit config to left gripper-v6

File: jsk_arc2017_baxter/robots/moveit_config/baxter.srdf.xacro (robot description, xacro)
@@ -1,13 +1,13 @@
 <?xml version="1.0" ?>
 <robot name="baxter" xmlns:xacro="http://www.ros.org/wiki/xacro">
-  <xacro:arg name="left_tip_name" default="left_gripper_vacuum_pad"/>
+  <xacro:arg name="left_tip_name" default="left_gripper_pad_with_base"/>
   <xacro:arg name="right_tip_name" default="right_gripper_pad_with_base"/>
   <xacro:include filename="$(find jsk_arc2017_baxter)/robots/moveit_config/baxter_base.srdf.xacro" />
   <xacro:baxter_base left_tip_name="$(arg left_tip_name)" right_tip_name="$(arg right_tip_name)"/>
   <!--Left End Effector Collisions-->
-  <xacro:include filename="$(find jsk_arc2017_baxter)/robots/moveit_config/left_vacuum_gripper.srdf.xacro" />
+  <xacro:include filename="$(find jsk_arc2017_baxter)/robots/moveit_config/vacuum_gripper.srdf.xacro" />
   <xacro:vacuum_gripper side="left"/>
   <!--Right End Effector Collisions-->
-  <xacro:include filename="$(find jsk_arc2017_baxter)/robots/moveit_config/right_vacuum_gripper.srdf.xacro" />
+  <xacro:include filename="$(find jsk_arc2017_baxter)/robots/moveit_config/vacuum_gripper.srdf.xacro" />
   <xacro:vacuum_gripper side="right"/>
 </robot>

File: jsk_arc2017_baxter/robots/moveit_config/baxter_base.srdf.xacro (robot description, xacro)
@@ -11,5 +11,5 @@
     <!--CHAINS: When a chain is specified, all the links along the chain (including endpoints) are included in the group. Additionally, all the joints that are parents to included links are also included. This means that joints along the chain and the parent joint of the base link are included in the group-->
     <!--SUBGROUPS: Groups can also be formed by referencing to already defined group names-->
-    <xacro:arg name="left_tip_name" default="left_gripper_vacuum_pad"/>
+    <xacro:arg name="left_tip_name" default="left_gripper_pad_with_base"/>
     <xacro:arg name="right_tip_name" default="right_gripper_pad_with_base"/>
     <group name="left_arm">
@@ -35,4 +35,5 @@
         <joint name="left_w1" value="1.26" />
         <joint name="left_w2" value="0" />
+        <joint name="left_gripper_prismatic_joint" value="0" />
         <joint name="left_gripper_vacuum_pad_joint" value="0" />
     </group_state>
